File: Pi-Game-Console.sch (KiCad schematic (older format))
At the start: 40 parts, among them J1 Micro_SD_Card, J2 HDMI_A, J3 Conn_Coaxial, J4 Conn_01x02_Female

Commit message: Ditching HDMI
Looks like we can't have DPI and HDMI enabled at the same time.  With that being the case, I'm not going to deal with all the components needed to add HDMI output.
Parts:
- removed J2: HDMI_A, Connector_HDMI:HDMI_A_Contact_Technology_HDMI-19APL2_Horizontal, symbol Connector:HDMI_A
Connections:
- net labels removed: HDMI_CEC, HDMI_CLK_N, HDMI_CLK_P, HDMI_D0_N, HDMI_D0_P, HDMI_D1_N, HDMI_D1_P, HDMI_D2_N, HDMI_D2_P, HDMI_HPD_N_1V8, HDMI_SCL, HDMI_SDA
- wire segments 180 -> 175
Changed lines of the file:
@@
-$EndComp
-$Comp
-L Connector:HDMI_A J2
-U 1 1 5E3B6A4F
-P 8700 3650
-F 0 "J2" H 9130 3696 50  0000 L CNN
-F 1 "HDMI_A" H 9130 3605 50  0000 L CNN
-F 2 "Connector_HDMI:HDMI_A_Contact_Technology_HDMI-19APL2_Horizontal" H 8725 3650 50  0001 C CNN
-F 3 "https://en.wikipedia.org/wiki/HDMI" H 8725 3650 50  0001 C CNN
-	1    8700 3650
-	1    0    0    -1
 $EndComp
 $Comp
@@
 	1    1400 2850
 	0    -1   -1   0
-$EndComp
-Text GLabel 6750 4300 2    50   Output ~ 0
-HDMI_CEC
-Text GLabel 6750 4600 2    50   Output ~ 0
-HDMI_SCL
-Text GLabel 6750 3100 2    50   Output ~ 0
-HDMI_CLK_P
-Text GLabel 6750 4450 2    50   Output ~ 0
-HDMI_SDA
-Text GLabel 6750 2950 2    50   Output ~ 0
-HDMI_CLK_N
-Text GLabel 6750 3400 2    50   Output ~ 0
-HDMI_D0_P
-Text GLabel 6750 3250 2    50   Output ~ 0
-HDMI_D0_N
-Text GLabel 6750 3700 2    50   Output ~ 0
-HDMI_D1_P
-Text GLabel 6750 3550 2    50   Output ~ 0
-HDMI_D1_N
-Text GLabel 6750 4000 2    50   Output ~ 0
-HDMI_D2_P
-Text GLabel 6750 3850 2    50   Output ~ 0
-HDMI_D2_N
-Text GLabel 8300 3750 0    50   Input ~ 0
-HDMI_CEC
-Text GLabel 8300 3950 0    50   Input ~ 0
-HDMI_SCL
-Text GLabel 8300 3450 0    50   Input ~ 0
-HDMI_CLK_P
-Text GLabel 8300 4050 0    50   Input ~ 0
-HDMI_SDA
-Text GLabel 8300 3550 0    50   Input ~ 0
-HDMI_CLK_N
-Text GLabel 8300 3250 0    50   Input ~ 0
-HDMI_D0_P
-Text GLabel 8300 3350 0    50   Input ~ 0
-HDMI_D0_N
-Text GLabel 8300 3050 0    50   Input ~ 0
-HDMI_D1_P
-Text GLabel 8300 3150 0    50   Input ~ 0
-HDMI_D1_N
-Text GLabel 8300 2850 0    50   Input ~ 0
-HDMI_D2_P
-Text GLabel 8300 2950 0    50   Input ~ 0
-HDMI_D2_N
-Text GLabel 8300 4350 0    50   Input ~ 0
-HDMI_HPD_N_1V8
-Text GLabel 6750 2650 2    50   Output ~ 0
-HDMI_HPD_N_1V8
-$Comp
-L power:+5V #PWR0104
-U 1 1 5E3E149F
-P 8700 2550
-F 0 "#PWR0104" H 8700 2400 50  0001 C CNN
-F 1 "+5V" H 8715 2723 50  0000 C CNN
-F 2 "" H 8700 2550 50  0001 C CNN
-F 3 "" H 8700 2550 50  0001 C CNN
-	1    8700 2550
-	1    0    0    -1
-$EndComp
-$Comp
-L power:GND #PWR0105
-U 1 1 5E3E1C78
-P 8900 4750
-F 0 "#PWR0105" H 8900 4500 50  0001 C CNN
-F 1 "GND" H 8905 4577 50  0000 C CNN
-F 2 "" H 8900 4750 50  0001 C CNN
-F 3 "" H 8900 4750 50  0001 C CNN
-	1    8900 4750
-	1    0    0    -1
 $EndComp
 Text GLabel 13100 2400 2    50   Output ~ 0
@@
 	0    -1   -1   0
 $EndComp
-Wire Wire Line
-	8900 4750 9000 4750
-Connection ~ 8900 4750
-Wire Wire Line
-	8500 4750 8600 4750
-Connection ~ 8600 4750
-Wire Wire Line
-	8600 4750 8700 4750
-Connection ~ 8700 4750
-Wire Wire Line
-	8700 4750 8800 4750
-Connection ~ 8800 4750
-Wire Wire Line
-	8800 4750 8900 4750
 $Comp
 L power:+5V #PWR0109

Commit message: Added usb gamepad and new hub
Parts:
- added C? (x2): 22pF, symbol Device:C_Small
- added C?: 0.1uF, symbol Device:C_Small
- added C?: 1uF, symbol Device:C_Small
- added C?: C_Small, symbol Device:C_Small
- added J?: FPC_Connector, symbol Connector:Conn_01x40_Female
- added J? (x2): Conn_01x04_Female, symbol Connector:Conn_01x04_Female
- added R?: 10k, symbol Device:R_Small
- added SW?: SW_DIP_x01, symbol Switch:SW_DIP_x01
- added SW? (x13): SW_Push, symbol Switch:SW_Push
- added U?: ATmega32U4-AU, Package_QFP:TQFP-44_10x10mm_P0.8mm, symbol MCU_Microchip_ATmega:ATmega32U4-AU
- added Y?: 16MHz, symbol Device:Crystal_Small
Connections:
- net +5V: now also C?.2, J?.1 (Pin_1), J?.1 (Pin_1), R?.1, SW?.2, U?.14 (VCC), U?.2 (UVCC), U?.24 (AVCC), U?.34 (VCC), U?.44 (AVCC), U?.7 (VBUS); no longer J4.1 (Pin_1)
- net GND: now also C?.1, C?.2, C?.2, C?.2, C?.2, J?.3 (Pin_3), J?.3 (Pin_3), SW?.2, SW?.2, SW?.2, SW?.2, SW?.2, SW?.2, SW?.2, SW?.2, SW?.2, SW?.2, SW?.2, SW?.2, SW?.2, U?.15 (GND), U?.23 (GND), U?.33 (~HWB~/PE2), U?.35 (GND), U?.43 (GND), U?.5 (UGND)
- net MCU_CONTROLLER_D_-: now reaches U?.27 (DM1)
- net MCU_CONTROLLER_D_-: now also U?.3 (D-)
- net MCU_CONTROLLER_D_+: now reaches U?.28 (DP1)
- net MCU_CONTROLLER_D_+: now also U?.4 (D+)
- new net: C?.1, U?.16 (XTAL2), Y?.1
- new net: C?.1, U?.17 (XTAL1), Y?.2
- new net: C?.1, U?.42 (AREF)
- new net: C?.1, U?.6 (UCAP)
- new net +BATT: J4.1 (Pin_1), SW?.1
- new net D_PAD_DOWN: SW?.1
- new net D_PAD_LEFT: SW?.1
- new net D_PAD_RIGHT: SW?.1
- new net D_PAD_UP: SW?.1
- new net GAMEPAD_A: SW?.1
- new net GAMEPAD_B: SW?.1
- new net GAMEPAD_HOME: SW?.1
- new net GAMEPAD_L: SW?.1
- new net GAMEPAD_R: SW?.1
- new net GAMEPAD_SELECT: SW?.1
- new net GAMEPAD_START: SW?.1
- new net GAMEPAD_X: SW?.1
- new net GAMEPAD_Y: SW?.1
- new net L_JOYSTICK_X: J?.2 (Pin_2), U?.36 (PF7)
- new net L_JOYSTICK_Y: J?.4 (Pin_4), U?.37 (PF6)
- new net MCU_MISO: U?.11 (PB3)
- new net MCU_MOSI: U?.10 (PB2)
- new net MCU_RESET: R?.2, U?.13 (~RESET)
- new net MCU_SCK: U?.9 (PB1)
- new net R_JOYSTICK_X: J?.2 (Pin_2), U?.38 (PF5)
- new net R_JOYSTICK_Y: J?.4 (Pin_4), U?.39 (PF4)
Other:
- moved on the sheet: J4

Commit message: Added HDMI and Audio Circuit
Still need to verify a few components for the HDMI connector.  Also, the Audio is only headphone out right now.  I still need to wire up the speaker and make it automaticaly switch.  Just need to do some research on audio jack styles.
Parts:
- removed MD?: Board_RPi_CM3lite_200pConnector_multipart, _, symbol KiCADinfo_RPi-modules:Board_RPi_CM3lite_200pConnector_multipart
- removed R?: 100k, symbol Device:R_Small
- added C? (x2): 10uF, symbol Device:C
- added C? (x2): 33nF, symbol Device:C
- added D? (x2): BAV99, Package_TO_SOT_SMD:SOT-23, symbol Diode:BAV99
- added J?: AudioJack3_Ground_SwitchTR, symbol Connector:AudioJack3_Ground_SwitchTR
- added LS?: Speaker, symbol Device:Speaker
- added R? (x2): R, symbol Device:R
- added R? (x2): 150R, symbol Device:R
- SW?: value SW_Push -> X_Button
- SW?: value SW_Push -> Y_Button
- SW?: value SW_Push -> B_Button
- SW?: value SW_Push -> A_Button
- SW?: value SW_Push -> L_Button
- SW?: value SW_Push -> R_Button
- SW?: value SW_Push -> Select_Button
- SW?: value SW_Push -> Start_Button
- SW?: value SW_Push -> D_PAD_LEFT_Button
- SW?: value SW_Push -> D_PAD_RIGHT_Button
- SW?: value SW_Push -> D_PAD_DOWN_Button
- SW?: value SW_Push -> D_PAD_UP_Button
- SW?: value SW_Push -> Home_Button
Connections:
- net +3V3: now also D?.2 (A), D?.2 (A)
- net D_PAD_DOWN: now also U?.22 (PD5)
- net D_PAD_LEFT: now also U?.26 (PD6)
- net D_PAD_RIGHT: now also U?.27 (PD7)
- net D_PAD_UP: now also U?.25 (PD4)
- net GAMEPAD_A: now also U?.18 (PD0)
- net GAMEPAD_B: now also U?.19 (PD1)
- net GAMEPAD_HOME: now also U?.29 (PB5)
- net GAMEPAD_L: now also U?.32 (PC7)
- net GAMEPAD_R: now also U?.31 (PC6)
- net GAMEPAD_SELECT: now also U?.30 (PB6)
- net GAMEPAD_START: now also U?.28 (PB4)
- net GAMEPAD_X: now also U?.20 (PD2)
- net GAMEPAD_Y: now also U?.21 (PD3)
- net GND: now also C?.2, C?.2, D?.1 (K), D?.1 (K), J?.G, J?.S, R?.1, R?.1
- net GPIO40: now reaches MD?.70 (GPIO40)
- net GPIO40: now also R?.1
- net GPIO45: now reaches MD?.84 (GPIO45)
- net GPIO45: now also R?.1
- new net: C?.1, C?.1, R?.2, R?.2 (x2)
- new net: C?.2, D?.3 (K), J?.R
- new net: C?.2, D?.3 (K), J?.T
- no-connect marks 27 -> 29
Other:
- note added: "Audio"
- moved on the sheet: J3, J?, MD?B, MD?E, MD?F, MD?G, R?

Commit message: Wired up the DPI display and Camera
Still need to wire up the DPI connector.
Parts:
- removed R? (x3): 100k, symbol Device:R_Small
- added J?: CAM1, symbol Connector_Generic:Conn_01x22
- added R?: 1k, symbol Device:R
- added R? (x2): 100k, symbol Device:R
- added R? (x2): 1.8k, symbol Device:R
Connections:
- net +3V3: now also J?.22 (Pin_22), R?.2, R?.2
- net GND: now also J1.6 (VSS), J?.1 (Pin_1), J?.10 (Pin_10), J?.13 (Pin_13), J?.16 (Pin_16), J?.19 (Pin_19), J?.4 (Pin_4), J?.7 (Pin_7), R?.1, R?.1, R?.2; no longer J1.9 (SHIELD)
- net GPIO45: now also R?.2
- net PI_USB_OTG_ID: now reaches MD?.168 (USB_OTGID)
- net PI_USB_OTG_ID: now also R?.1
- net CAM1_D3_P: now reaches MD?.135 (CAM1_DP3)
- net CAM1_D3_P: now also J?.14 (Pin_14)
- net CAM1_D3_N: now reaches MD?.137 (CAM1_DN3)
- net CAM1_D3_N: now also J?.15 (Pin_15)
- net CAM1_D2_P: now reaches MD?.141 (CAM1_DP2)
- net CAM1_D2_P: now also J?.11 (Pin_11)
- net CAM1_D2_N: now reaches MD?.143 (CAM1_DN2)
- net CAM1_D2_N: now also J?.12 (Pin_12)
- net CAM1_C_P: now reaches MD?.147 (CAM1_CP)
- net CAM1_C_P: now also J?.9 (Pin_9)
- net CAM1_C_N: now reaches MD?.149 (CAM1_CN)
- net CAM1_C_N: now also J?.8 (Pin_8)
- net CAM1_D1_P: now reaches MD?.153 (CAM1_DP1)
- net CAM1_D1_P: now also J?.5 (Pin_5)
- net CAM1_D1_N: now reaches MD?.155 (CAM1_DN1)
- net CAM1_D1_N: now also J?.6 (Pin_6)
- net CAM1_D0_P: now reaches MD?.159 (CAM1_DP0)
- net CAM1_D0_P: now also J?.2 (Pin_2)
- net CAM1_D0_N: now reaches MD?.161 (CAM1_DN0)
- net CAM1_D0_N: now also J?.3 (Pin_3)
- net DISP_H_SYNC: now reaches MD?.11 (GPIO3)
- net DISP_B0: now reaches MD?.15 (GPIO4)
- net DISP_B1: now reaches MD?.17 (GPIO5)
- net DISP_B2: now reaches MD?.21 (GPIO6)
- net DISP_B3: now reaches MD?.23 (GPIO7)
- net DISP_B4: now reaches MD?.27 (GPIO8)
- net CD1_SDA: now reaches MD?.28 (GPIO28)
- net CD1_SDA: now also J?.21 (Pin_21), R?.1
- net DISP_B5: now reaches MD?.29 (GPIO9)
- net DISP_CLK: now reaches MD?.3 (GPIO0)
- net CD1_SCL: now reaches MD?.30 (GPIO29)
- net CD1_SCL: now also J?.20 (Pin_20), R?.1
- net DISP_B6: now reaches MD?.33 (GPIO10)
- net CAM1_IO1: now reaches MD?.34 (GPIO30)
- net CAM1_IO1: now also J?.18 (Pin_18)
- net DISP_B7: now reaches MD?.35 (GPIO11)
- net CAM1_IO0: now reaches MD?.36 (GPIO31)
- net CAM1_IO0: now also J?.17 (Pin_17)
- net DISP_G0: now reaches MD?.45 (GPIO12)
- net DISP_G1: now reaches MD?.47 (GPIO13)
- net DISP_DE: now reaches MD?.5 (GPIO1)
- net DISP_G2: now reaches MD?.51 (GPIO14)
- net DISP_G3: now reaches MD?.53 (GPIO15)
- net DISP_G4: now reaches MD?.57 (GPIO16)
- net DISP_G5: now reaches MD?.59 (GPIO17)
- net DISP_G6: now reaches MD?.63 (GPIO18)
- net DISP_G7: now reaches MD?.65 (GPIO19)
- net DISP_R0: now reaches MD?.69 (GPIO20)
- net DISP_R1: now reaches MD?.71 (GPIO21)
- net DISP_R2: now reaches MD?.75 (GPIO22)
- net DISP_R3: now reaches MD?.77 (GPIO23)
- net DISP_R4: now reaches MD?.81 (GPIO24)
- net DISP_R5: now reaches MD?.83 (GPIO25)
- net DISP_R6: now reaches MD?.87 (GPIO26)
- net DISP_R7: now reaches MD?.89 (GPIO27)
- net DISP_V_SYNC: now reaches MD?.9 (GPIO2)
- new net GPIO44: R?.2
- no-connect marks 29 -> 35
Other:
- moved on the sheet: J1, MD?F
