File: Pi-Game-Console.sch (KiCad schematic (older format))
At the start: 77 parts, among them J1 Micro_SD_Card, J3 Conn_Coaxial, J4 Conn_01x02_Female

Commit message: Added USB Ports and wired up more of the DPI connector
Parts:
- added J? (x2): USB_A, symbol Connector:USB_A
- C1, C10, C11, C12, C13, C14, C15, C17, C18, C2, C3, C4, C5, C6, C7, C8, C9: renamed from C?; footprint (none) -> Capacitor_SMD:C_0805_2012Metric
- C16: renamed from C?; footprint (none) -> Connector_HDMI:HDMI_Micro-D_Molex_46765-2x0x
- F1, F2: renamed from F?; footprint (none) -> Diode_SMD:Littelfuse_PolyZen-LS
- J2: renamed from J?; footprint (none) -> Connector_FFC-FPC:Hirose_FH12-22S-0.5SH_1x22-1MP_P0.50mm_Horizontal
- J5: renamed from J?; footprint (none) -> Connector_Audio:Jack_3.5mm_PJ31060-I_Horizontal
- J6: renamed from J?; footprint (none) -> Connector_FFC-FPC:Hirose_FH12-40S-0.5SH_1x40-1MP_P0.50mm_Horizontal
- J7, J8: renamed from J?; footprint (none) -> Connector_Molex:Molex_CLIK-Mate_502585-0470_1x04-1MP_P1.50mm_Horizontal
- L1: renamed from L?; footprint (none) -> Inductor_SMD:L_6.3x6.3_H3
- LS1: renamed from LS?; footprint (none) -> Connector_Molex:Molex_CLIK-Mate_502382-0270_1x02-1MP_P1.25mm_Vertical
- MD1: renamed from MD?; footprint _ -> footprints:Conn_TE-DDR2-SODIMM-0.6-200P-doublesided
- R1, R10, R11, R12, R13, R14, R15, R16, R17, R18, R2, R3, R4, R5, R6, R7, R8, R9: renamed from R?; footprint (none) -> Resistor_SMD:R_0805_2012Metric
- SW1: renamed from SW?; footprint (none) -> Button_Switch_THT:SW_CuK_OS102011MA1QN1_SPDT_Angled
- SW10, SW11, SW12, SW13, SW14, SW15, SW2, SW3, SW4, SW5, SW6, SW7, SW8, SW9: renamed from SW?; footprint (none) -> Button_Switch_SMD:SW_Push_1P1T_NO_6x6mm_H9.5mm
- U1, U3: renamed from U?; footprint (none) -> Package_SO:SOIC-28W_7.5x17.9mm_P1.27mm
- Y1, Y2, Y3: renamed from Y?; footprint (none) -> Crystal:Crystal_SMD_ECS_CSM3X-2Pin_7.6x4.1mm
- gave numbers to parts that had none: 3
Connections:
- net +3V3: now also J6.4 (Pin_4)
- net +5V: now also J?.1 (VBUS), J?.1 (VBUS)
- net DISP_B0: now also J6.21 (Pin_21)
- net DISP_B1: now also J6.22 (Pin_22)
- net DISP_B2: now also J6.23 (Pin_23)
- net DISP_B3: now also J6.24 (Pin_24)
- net DISP_B4: now also J6.25 (Pin_25)
- net DISP_B5: now also J6.26 (Pin_26)
- net DISP_B6: now also J6.27 (Pin_27)
- net DISP_B7: now also J6.28 (Pin_28)
- net DISP_CLK: now also J6.30 (Pin_30)
- net DISP_DE: now also J6.34 (Pin_34)
- net DISP_G0: now also J6.13 (Pin_13)
- net DISP_G1: now also J6.14 (Pin_14)
- net DISP_G2: now also J6.15 (Pin_15)
- net DISP_G3: now also J6.16 (Pin_16)
- net DISP_G4: now also J6.17 (Pin_17)
- net DISP_G5: now also J6.18 (Pin_18)
- net DISP_G6: now also J6.19 (Pin_19)
- net DISP_G7: now also J6.20 (Pin_20)
- net DISP_H_SYNC: now also J6.32 (Pin_32)
- net DISP_R0: now also J6.5 (Pin_5)
- net DISP_R1: now also J6.6 (Pin_6)
- net DISP_R2: now also J6.7 (Pin_7)
- net DISP_R3: now also J6.8 (Pin_8)
- net DISP_R4: now also J6.9 (Pin_9)
- net DISP_R5: now also J6.10 (Pin_10)
- net DISP_R6: now also J6.11 (Pin_11)
- net DISP_R7: now also J6.12 (Pin_12)
- net DISP_V_SYNC: now also J6.33 (Pin_33)
- net GND: now also J6.29 (Pin_29), J6.3 (Pin_3), J6.36 (Pin_36), J?.4 (GND), J?.4 (GND), J?.5 (Shield), J?.5 (Shield)
- net MCU_CONTROLLER_D_+: now also U1.10 (DM1)
- net MCU_CONTROLLER_D_-: now also U1.11 (DP1)
- net USB2_D_-: now reaches U1.4 (DM4)
- net USB2_D_-: now also J?.2 (D-)
- net USB2_D_+: now reaches U1.5 (DP4)
- net USB2_D_+: now also J?.3 (D+)
- net USB3_D_-: now reaches U1.6 (DM3)
- net USB3_D_-: now also J?.2 (D-)
- net USB3_D_+: now reaches U1.7 (DP3)
- net USB3_D_+: now also J?.3 (D+)
Other:
- moved on the sheet: J6

Commit message: Cleaned up schematic
Parts:
- added C20, C26: 10uF, symbol Device:C
- added C21, C22: C_Small, symbol Device:C_Small
- added C23, C24: 1uF, symbol Device:C
- added C25: 0.1uF, symbol Device:C
- added D10: MBR0540, symbol Device:D
- added D11: MM3Z24VT1G, symbol Device:D
- added D8: 1N4148, symbol Device:D
- added D9: LED, symbol Device:LED
- added FB? (x4): Ferrite_Bead_Small, symbol Device:Ferrite_Bead_Small
- added JP1, JP2, JP3: SolderJumper_2_Open, symbol Jumper:SolderJumper_2_Open
- added L2: 6.8uH power L CID 2276, symbol Device:L
- added R22, R23: 20k, symbol Device:R
- added R24, R25, R27: 127, symbol Device:R
- added R26: 67, symbol Device:R
- added R28: 10k, symbol Device:R
- added R29: 470, symbol Device:R
- added RN? (x7): R_Pack04, symbol Device:R_Pack04
- added RV1: R_POT, symbol Device:R_POT
- added TP1: JTAG_TRST_N, symbol Connector:TestPoint
- added TP2: JTAG_TDI, symbol Connector:TestPoint
- added TP3: JTAG_TMS, symbol Connector:TestPoint
- added TP4: JTAG_TDO, symbol Connector:TestPoint
- added TP5: JTAG_TCK, symbol Connector:TestPoint
- added U4: FAN5333BSX, symbol Pi_USB:FAN5333BSX
- added U5: AR1100, symbol Pi_USB:AR1100
- added Y4: 12MHz, Crystal:Crystal_SMD_ECS_CSM3X-2Pin_7.6x4.1mm, symbol Device:Crystal_Small
- J10, J11: renamed from J?; footprint (none) -> Connector_USB:USB_A_Stewart_SS-52100-001_Horizontal
Connections:
- net +3V3: now also R22.1
- net +5V: now also C20.1, L2.1, R23.1, U4.5 (VIN), U5.1 (VDD), U5.4 (MODE)
- net DISP_B0: now also RN?.1 (R1.1); no longer J6.21 (Pin_21)
- net DISP_B1: now also RN?.2 (R2.1); no longer J6.22 (Pin_22)
- net DISP_B2: now also RN?.3 (R3.1); no longer J6.23 (Pin_23)
- net DISP_B3: now also RN?.4 (R4.1); no longer J6.24 (Pin_24)
- net DISP_B4: now also RN?.1 (R1.1); no longer J6.25 (Pin_25)
- net DISP_B5: now also RN?.2 (R2.1); no longer J6.26 (Pin_26)
- net DISP_B6: now also RN?.3 (R3.1); no longer J6.27 (Pin_27)
- net DISP_B7: now also RN?.4 (R4.1); no longer J6.28 (Pin_28)
- net DISP_CLK: now also RN?.1 (R1.1); no longer J6.30 (Pin_30)
- net DISP_DE: now also RN?.4 (R4.1); no longer J6.34 (Pin_34)
- net DISP_G0: now also RN?.1 (R1.1); no longer J6.13 (Pin_13)
- net DISP_G1: now also RN?.2 (R2.1); no longer J6.14 (Pin_14)
- net DISP_G2: now also RN?.3 (R3.1); no longer J6.15 (Pin_15)
- net DISP_G3: now also RN?.4 (R4.1); no longer J6.16 (Pin_16)
- net DISP_G4: now also RN?.1 (R1.1); no longer J6.17 (Pin_17)
- net DISP_G5: now also RN?.2 (R2.1); no longer J6.18 (Pin_18)
- net DISP_G6: now also RN?.3 (R3.1); no longer J6.19 (Pin_19)
- net DISP_G7: now also RN?.4 (R4.1); no longer J6.20 (Pin_20)
- net DISP_H_SYNC: now also RN?.2 (R2.1); no longer J6.32 (Pin_32)
- net DISP_R0: now also RN?.1 (R1.1); no longer J6.5 (Pin_5)
- net DISP_R1: now also RN?.2 (R2.1); no longer J6.6 (Pin_6)
- net DISP_R2: now also RN?.3 (R3.1); no longer J6.7 (Pin_7)
- net DISP_R3: now also RN?.4 (R4.1); no longer J6.8 (Pin_8)
- net DISP_R4: now also RN?.1 (R1.1); no longer J6.9 (Pin_9)
- net DISP_R5: now also RN?.2 (R2.1); no longer J6.10 (Pin_10)
- net DISP_R6: now also RN?.3 (R3.1); no longer J6.11 (Pin_11)
- net DISP_R7: now also RN?.4 (R4.1); no longer J6.12 (Pin_12)
- net DISP_V_SYNC: now also RN?.3 (R3.1); no longer J6.33 (Pin_33)
- net GND: now also C20.2, C21.2, C22.2, C23.2, C24.2, C25.2, C26.1, JP1.2 (B), JP2.2 (B), JP3.2 (B), R24.2, R29.2, U4.2 (SHDNGND), U5.13 (SX-), U5.20 (VSS), U5.6 ((Y+)), U5.8 (SY-), U5.9 (SX+)
- net MCU_CONTROLLER_D_+: now also U1.11 (DP1); no longer U1.10 (DM1)
- net MCU_CONTROLLER_D_-: now also U1.10 (DM1); no longer U1.11 (DP1)
- net at MD1.172 (VC_TRST_N): now also TP1.1
- net at MD1.174 (VC_TDI): now also TP2.1
- net at MD1.176 (VC_TMS): now also TP3.1
- net at MD1.178 (VC_TDO): now also TP4.1
- net at MD1.180 (VC_TCK): now also TP5.1
- net DISP_LED_K: now reaches J6.1 (Pin_1)
- net DISP_LED_K: now also C25.1, D11.2 (A), R24.1, R25.1, R26.1, R27.1, U4.3 (FB)
- net +24V: now reaches J6.2 (Pin_2)
- net +24V: now also C23.1, C24.1, D10.1 (K), D11.1 (K)
- net at J6.31 (Pin_31): now also R22.2
- net at J6.37 (Pin_37): now also FB?.1
- net at J6.38 (Pin_38): now also FB?.1
- net at J6.39 (Pin_39): now also FB?.1
- net at J6.40 (Pin_40): now also FB?.1
- net TOUCH_USB_D_-: now reaches U1.8 (DM2)
- net TOUCH_USB_D_-: now also U5.18 (D-)
- net TOUCH_USB_D_+: now reaches U1.9 (DP2)
- net TOUCH_USB_D_+: now also U5.19 (D+)
- net USB2_D_+ renamed USB0_D_+
- net USB2_D_- renamed USB0_D_-
- net USB3_D_+ renamed USB1_D_+
- net USB3_D_- renamed USB1_D_-
- new net: J6.10 (Pin_10), RN?.7 (R2.2)
- new net: J6.11 (Pin_11), RN?.6 (R3.2)
- new net: J6.12 (Pin_12), RN?.5 (R4.2)
- new net: J6.13 (Pin_13), RN?.8 (R1.2)
- new net: J6.14 (Pin_14), RN?.7 (R2.2)
- new net: J6.15 (Pin_15), RN?.6 (R3.2)
- new net: J6.16 (Pin_16), RN?.5 (R4.2)
- new net: J6.17 (Pin_17), RN?.8 (R1.2)
- new net: J6.18 (Pin_18), RN?.7 (R2.2)
- new net: J6.19 (Pin_19), RN?.6 (R3.2)
- new net: J6.20 (Pin_20), RN?.5 (R4.2)
- new net: J6.21 (Pin_21), RN?.8 (R1.2)
- new net: J6.22 (Pin_22), RN?.7 (R2.2)
- new net: J6.23 (Pin_23), RN?.6 (R3.2)
- new net: J6.24 (Pin_24), RN?.5 (R4.2)
- new net: J6.25 (Pin_25), RN?.8 (R1.2)
- new net: J6.26 (Pin_26), RN?.7 (R2.2)
- new net: J6.27 (Pin_27), RN?.6 (R3.2)
- new net: J6.28 (Pin_28), RN?.5 (R4.2)
- new net: J6.30 (Pin_30), RN?.8 (R1.2)
- new net: J6.32 (Pin_32), RN?.7 (R2.2)
- new net: J6.33 (Pin_33), RN?.6 (R3.2)
- new net: J6.34 (Pin_34), RN?.5 (R4.2)
- new net: J6.5 (Pin_5), RN?.8 (R1.2)
- new net: J6.6 (Pin_6), RN?.7 (R2.2)
- new net: J6.7 (Pin_7), RN?.6 (R3.2)
- new net: J6.8 (Pin_8), RN?.5 (R4.2)
- new net: J6.9 (Pin_9), RN?.8 (R1.2)
- new net: D10.2 (A), L2.2, U4.1 (SW)
- new net: D8.2 (A), R23.2, U4.4 (PWM)
- new net: JP1.1 (A), R25.2
- new net: JP2.1 (A), R26.2
- new net: JP3.1 (A), R27.2
- new net: R28.2, U5.11 (WAKE)
- new net: C26.2, U5.17 (VUSB)
- new net: C21.1, U5.2 (OSC1), Y4.2
- new net: C22.1, U5.3 (OSC2), Y4.1
- new net: D9.2 (A), U5.5 (LED)
- new net: D9.1 (K), R29.1
- new net DISP_X_+: FB?.2, U5.7 (X+)
- new net DISP_X_-: FB?.2, R28.1, U5.14 (X-)
- new net DISP_Y_+: FB?.2, U5.15 (Y+)
- new net DISP_Y_-: FB?.2, U5.16 (Y-)
Other:
- note added: "Button inputs for Joysticks or second L/R buttons?"
- note added: "Camera"
- note added: "DSI Pins\n(Not used)"
- note added: "Display"
- note added: "I have two different USB hub ICs. I'm not sure which one I want to use yet.\nThe one on the right has more components, but isn't as fast."
- note added: "Power Connections"
- note added: "Replace this with a single pot? (no soldered jumpers)"
- note added: "SD Card"
- note added: "USB Hub"
- note added: "USB Xinput Device"
- moved on the sheet: C1, C10, C11, C12, C2, C3, C4, C8, C9, D1, D2, J1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

Commit message: Added documentation
Parts:
- gave numbers to parts that had none: 11
- renumbered C25 to C10, C26 to C11, C5 to C12, C6 to C13, C7 to C14, C8 to C15, C9 to C16, C10 to C17, C11 to C18, C12 to C19, C13 to C20, C14 to C21, C15 to C22, C16 to C23, C17 to C24, C18 to C25, C20 to C3, C3 to C4, C21 to C5, C22 to C6, C4 to C7, C23 to C8, C24 to C9, D8 to D3, D9 to D4, D10 to D5, D11 to D6, J4 to J1, J8 to J10, J5 to J2, J6 to J3, J3 to J4, J1 to J5, J2 to J6, J10 to J7, J11 to J8, J7 to J9, L2 to L1, L1 to L2, R7 to R10, R8 to R11, R24 to R12, R25 to R13, R26 to R14, R27 to R15, R28 to R16, R9 to R17, R10 to R18, R11 to R19, R12 to R20, R13 to R21, R14 to R22, R15 to R23, R16 to R24, R17 to R25, R18 to R26, R22 to R5, R5 to R6, R23 to R7, R6 to R8, R29 to R9, U4 to U1, U5 to U2, U1 to U3, U2 to U4, U3 to U5, Y4 to Y1, Y1 to Y2, Y2 to Y3, Y3 to Y4
Other:
- note added: "Backlight Driver"
- note added: "HDMI Out"
- note added: "Touchscreen Driver"
- note added: "might ditch both this and the camera connector"
- note added: "update this to use the Retro CM3 Audio circuit"

Commit message: Switched Audio Circuit to use Retro-CM3 Schematic
Parts:
- removed C1, C2: 10uF, Capacitor_SMD:C_0805_2012Metric, symbol Device:C
- removed C4, C7: 33nF, Capacitor_SMD:C_0805_2012Metric, symbol Device:C
- removed D1, D2: BAV99, Package_TO_SOT_SMD:SOT-23, symbol Diode:BAV99
- removed J2: AudioJack3_Ground_SwitchTR, Connector_Audio:Jack_3.5mm_PJ31060-I_Horizontal, symbol Connector:AudioJack3_Ground_SwitchTR
- removed R10, R11: R, Resistor_SMD:R_0805_2012Metric, symbol Device:R
- removed R6, R8: 150R, Resistor_SMD:R_0805_2012Metric, symbol Device:R
- added C? (x5): 100nF, symbol Device:C
- added C? (x2): 47uF, symbol Device:C
- added C?: 10uF, symbol Device:C
- added C?: 100uF, symbol Device:C
- added J?: AudioJack3_Ground_SwitchTR, symbol Connector:AudioJack3_Ground_SwitchTR
- added R? (x2): 220, symbol Device:R
- added R? (x4): 4.7, symbol Device:R
- added R? (x2): 1.8k, symbol Device:R
- added R?: 10k, symbol Device:R
- added U?: NC7WZ16, symbol Pi_USB:NC7WZ16
- added U?: TDA2822, symbol Pi_USB:TDA2822
Connections:
- net +3V3: now also U?.5 (VCC)
- net +5V: now also C?.2, U?.2 (VCC)
- net GND: now also C?.1, C?.1, C?.1, C?.2, C?.2, C?.2, J?.G, J?.S, R?.1, R?.1, R?.2, R?.2, R?.2, U?.2 (GND), U?.4 (GND), U?.6 (Input2)
- net GPIO44: now also MD1.82 (GPIO44)
- net AUDIO_PWM_1: now reaches MD1.72 (GPIO41)
- net AUDIO_PWM_1: now also U?.3 (A2)
- net at LS1.1: now also R?.2, U?.1 (OUTPUT1)
- net at LS1.2: now also R?.2, U?.3 (OUTPUT2)
- net GPIO40 renamed AUDIO_PWM_0
- net AUDIO_PWM_0: now also U?.1 (A1)
- new net: R?.1, U?.4 (Y2)
- new net: R?.2, U?.6 (Y1)
- new net: C?.2, C?.2, R?.1, R?.1
- new net: C?.1, C?.2, R?.2, R?.2
- new net: C?.1, C?.2, U?.5 (NP2)
- new net: C?.1, U?.8 (NP1)
- new net: C?.2, R?.1
- new net: C?.1, R?.1
- new net AUDIO_L_OUT: C?.1, J?.T, R?.2
- new net AUDIO_R_OUT: C?.1, J?.R, R?.1
- new net SPEAKER: J?.TN, R?.1, U?.7 (Input1)
- no-connect marks 35 -> 33
Other:
- note removed: "update this to use the Retro CM3 Audio circuit"
- moved on the sheet: LS1

Commit message: Removed Second USB Hub
Also wired up a few more connections.
Parts:
- removed C20: 1u, Capacitor_SMD:C_0805_2012Metric, symbol Device:C_Small
- removed C21, C22: 100n, Capacitor_SMD:C_0805_2012Metric, symbol Device:C_Small
- removed C23: 100n, Connector_HDMI:HDMI_Micro-D_Molex_46765-2x0x, symbol Device:C_Small
- removed C24, C25: 33p, Capacitor_SMD:C_0805_2012Metric, symbol Device:C_Small
- removed F2: Polyfuse_Small, Diode_SMD:Littelfuse_PolyZen-LS, symbol Device:Polyfuse_Small
- removed L2: 47u, Inductor_SMD:L_6.3x6.3_H3, symbol Device:L_Small
- removed R20: 100, Resistor_SMD:R_0805_2012Metric, symbol Device:R_Small
- removed R21, R23, R26: 10k, Resistor_SMD:R_0805_2012Metric, symbol Device:R_Small
- removed R22: 680, Resistor_SMD:R_0805_2012Metric, symbol Device:R_Small
- removed R24: 100k, Resistor_SMD:R_0805_2012Metric, symbol Device:R_Small
- removed R25: 5.1k, Resistor_SMD:R_0805_2012Metric, symbol Device:R_Small
- removed SW2: SW_RST, Button_Switch_SMD:SW_Push_1P1T_NO_6x6mm_H9.5mm, symbol Switch:SW_Push
- removed U5: GL850G, Package_SO:SOIC-28W_7.5x17.9mm_P1.27mm, symbol USB_Hub-cache:GL850G
- removed Y4: 12Mhz, Crystal:Crystal_SMD_ECS_CSM3X-2Pin_7.6x4.1mm, symbol Device:Crystal
- added C15: 10uF, symbol Device:C
- added R1: 100k, symbol Device:R
- gave numbers to parts that had none: 21
- renumbered C5 to C11, C6 to C12, C8 to C13, C9 to C14, C11 to C16, C10 to C17, C15 to C18, C16 to C19, C17 to C20, C18 to C21, C19 to C22, C12 to C23, C13 to C24, C14 to C25, C3 to C6, D3 to D1, D4 to D2, D5 to D3, D6 to D4, J3 to J2, J4 to J3, R7 to R14, R9 to R17, R12 to R18, R13 to R19, R1 to R2, R14 to R20, R15 to R21, R16 to R22, R18 to R23, R19 to R24, R17 to R25, R2 to R3, R3 to R4, R4 to R5, R5 to R6, SW11 to SW10, SW12 to SW11, SW13 to SW12, SW14 to SW13, SW15 to SW14, SW3 to SW2, SW4 to SW3, SW5 to SW4, SW6 to SW5, SW7 to SW6, SW8 to SW7, SW9 to SW8, SW10 to SW9, U1 to U3, U2 to U4, U4 to U5, U3 to U6, Y3 to Y2, Y2 to Y3
Connections:
- net +3V3: now also J5.4 (VDD), MD1.4 (SDX_VDD), MD1.6 (SDX_VDD), C15.1, R1.2; no longer MD1.2 (EMMC_DISABLE_N)
- net GND: now also C15.2
- new net: MD1.2 (EMMC_DISABLE_N), R1.1
- no-connect marks 33 -> 31
Other:
- note removed: "?"
- note removed: "I have two different USB hub ICs. I'm not sure which one I want to use yet.\nThe one on the right has more components, but isn't as fast."
- note removed: "Switch to FE1.1s?"
- moved on the sheet: C1, C10, C13, C14, C17, C2, C23, C24, C25, C3, C4, C5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

Commit message: Updated the audio generation to use I2S
Parts:
- removed C4, C5: 100nF, symbol Device:C
- removed C7, C8: 47uF, symbol Device:C
- removed J4: AudioJack3_Ground_SwitchTR, symbol Connector:AudioJack3_Ground_SwitchTR
- removed R10, R11: 4.7, symbol Device:R
- removed R15, R16: 1.8k, symbol Device:R
- removed R8, R9: 220, symbol Device:R
- removed U1: NC7WZ16, symbol Pi_USB:NC7WZ16
- added C? (x2): 0.1uF, symbol Device:C_Small
- added C? (x2): 10uF, symbol Device:C_Small
- added C? (x2): 47uF, symbol Device:C_Small
- added C? (x2): 0.01uF, symbol Device:C_Small
- added FB? (x2): Ferrite, symbol Device:Ferrite_Bead_Small
- added J?: AudioJack3_Ground_SwitchTR, symbol Connector:AudioJack3_Ground_SwitchTR
- added R? (x2): 220k, symbol Device:R
- added R? (x2): 100, symbol Device:R
- added U?: UDA1334A, Package_SO:SSOP-16_4.4x5.2mm_P0.65mm, symbol Audio:UDA1334ATS
Connections:
- net +3V3: now also FB?.2, U?.4 (VDDD)
- net CAM1_IO0: now also MD1.76 (GPIO42); no longer MD1.36 (GPIO31)
- net CAM1_IO1: now also MD1.78 (GPIO43); no longer MD1.34 (GPIO30)
- net CD1_SCL: now also MD1.84 (GPIO45); no longer MD1.30 (GPIO29)
- net CD1_SDA: now also MD1.82 (GPIO44); no longer MD1.28 (GPIO28)
- net GND: now also C?.1, C?.1, C?.2, FB?.1, J?.G, U?.10 (PLL0), U?.11 (SFOR0), U?.5 (VSSD), U?.6 (SYSCLK/PLL1), U?.7 (SFOR1), U?.9 (DEEM/CLKOUT)
- net SPEAKER: now also J?.TN
- net AUDIO_PWM_0: no longer names the net of MD1.70 (GPIO40)
- net AUDIO_PWM_1: no longer names the net of MD1.72 (GPIO41)
- net GPIO44 renamed AUDIO_BIT_CLK
- net AUDIO_BIT_CLK: now also MD1.28 (GPIO28), U?.1 (BCK); no longer MD1.82 (GPIO44)
- net GPIO45 renamed AUDIO_LR_CLK
- net AUDIO_LR_CLK: now also MD1.30 (GPIO29), U?.2 (WS); no longer MD1.84 (GPIO45)
- new net: C?.1, C?.1, U?.12 (Vref(DAC))
- new net: C?.2, C?.2, FB?.1, U?.13 (VDDA)
- new net: C?.2, U?.14 (VOUTL)
- new net: C?.2, U?.16 (VOUTR)
- new net: C?.1, R?.2, R?.2
- new net: C?.1, R?.1, R?.1
- new net AUDIO_DATA_IN: MD1.36 (GPIO31), U?.3 (DATAI)
- new net AUDIO_OUT_L: C?.2, J?.T, R?.1
- new net AUDIO_OUT_R: C?.1, J?.R, R?.2
- new net GNDA: C?.1, C?.2, C?.2, FB?.2, J?.S, R?.1, R?.2, U?.15 (VSSA)
Other:
- note added: "I2S Audio DAC"
- note added: "Speaker Amp"
