File: Pi-Game-Console.kicad_pcb (KiCad board)
At the start: 2 copper layers, 119 parts, among them J1 Conn_01x02_Female, J10 Conn_01x04_Female, J11 2001-1-2-21-00-BK, J2 FPC_Connector, J3 Conn_Coaxial, J4 AudioJack3_Ground_SwitchTR, J5 Micro_SD_Card, J6 CAM1, J7 USB_A, J8 USB_A, J9 Conn_01x04_Female, Q1 2N7002P.215, SW1 SW_DIP_x01, SW10 Y_Button, SW11 D_PAD_UP_Button, SW12 D_PAD_DOWN_Button, SW13 D_PAD_LEFT_Button, SW14 D_PAD_RIGHT_Button, SW2 Home_Button, SW3 Start_Button, SW4 Select_Button, SW5 L_Button, SW6 R_Button, SW7 A_Button, SW8 B_Button, SW9 X_Button, U1 UDA1334ATS, U2 TDA2822, U3 FAN5333BSX, U4 AR1100, U5 ATmega32U4-AU, U6 FE1.1s, Y1 12MHz, Y2 16MHz, Y3 12MHz

Commit message: updated display traces.
Parts:
- J11: moved to B.Cu
- moved J11 95.4 mm to (-22.9, 142.2), turned to 90 degrees
- moved J6 9.40 mm to (-3.05, 127.0)
Routing:
- net DISP_DE: track 0.00 -> 36.0 mm, vias 0 -> 2
- net DISP_V_SYNC: track 0.00 -> 33.9 mm, vias 0 -> 2
- net DISP_CLK: track 0.00 -> 33.4 mm, vias 0 -> 2
- net DISP_H_SYNC: track 0.00 -> 32.4 mm, vias 0 -> 2
- net DISP_B3: track 0.00 -> 24.2 mm, vias 0 -> 2
- net DISP_B5: track 0.00 -> 24.0 mm, vias 0 -> 2
- net DISP_B7: track 0.00 -> 23.5 mm, vias 0 -> 2
- net DISP_B2: track 0.00 -> 21.9 mm, vias 0 -> 2
- net DISP_B4: track 0.00 -> 21.2 mm, vias 0 -> 2
- net DISP_B6: track 0.00 -> 20.9 mm, vias 0 -> 2
- net DISP_B1: track 2.79 -> 23.5 mm, vias 1 -> 2

Commit message: Fixed footprints, added PWM to display backlight
Parts:
- added RV2: R_POT, Potentiometer_SMD:Potentiometer_Bourns_3269P_Horizontal, F.Cu at (135.9, 186.7)
- J10, J9: value Conn_01x04_Female -> Conn_01x05_Female; footprint Connector_Molex:Molex_CLIK-Mate_502585-0470_1x04-1MP_P1.50mm_Horizontal -> Connector_FFC-FPC:Molex_200528-0050_1x05-1MP_P1.00mm_Horizontal
- J11: footprint Connector_HDMI:HDMI_Micro-D_Molex_46765-2x0x -> HDMI_MOLEX:HDMI_MOLEX_471510001
- SW10, SW11, SW12, SW13, SW14, SW2, SW3, SW4, SW5, SW6, SW7, SW8, SW9: footprint Button_Switch_SMD:SW_Push_1P1T_NO_6x6mm_H9.5mm -> Button_Switch_THT:SW_PUSH_6mm_H5mm
- moved J5 117.6 mm to (54.6, 170.2), turned to 90 degrees
- moved J3 14.5 mm to (-36.8, 123.2)
- moved J10 6.35 mm to (193.0, 171.4), turned to 0 degrees
- moved J9 3.81 mm to (116.8, 171.4), turned to 0 degrees
- moved SW11 2.84 mm to (130.8, 147.3)
- moved SW12 2.84 mm to (130.8, 162.6)
- moved SW13 2.84 mm to (123.2, 154.9)
- moved SW14 2.84 mm to (138.4, 154.9)
- moved J11 2.54 mm to (-22.9, 139.7)
- renumbered D2 to D1, D3 to D2, D4 to D3, D5 to D4, D6 to D5, D7 to D6, D8 to D7, D9 to D8, JP3 to JP2, R15 to R14, R16 to R15, R17 to R16, R19 to R17, R20 to R18, R21 to R19, R22 to R20, R23 to R21, R24 to R22, R25 to R23, R26 to R24
Connections:
- D1 pad 1: Net-(D2-Pad1) -> Net-(D1-Pad1)
- D1 pad 2: Net-(D2-Pad2) (its old number) -> Net-(D1-Pad2)
- JP2 pad 1: Net-(JP3-Pad1) -> Net-(JP2-Pad1)
- R14 pad 1: Net-(D2-Pad1) -> Net-(D1-Pad1)
- R17 pad 2: Net-(JP3-Pad1) -> Net-(JP2-Pad1)
- U3 pad 4: Net-(D1-Pad2) -> DISP_PWM
- U4 pad 5: Net-(D2-Pad2) (its old number) -> Net-(D1-Pad2)
- U5 pad 12: Net-(U5-Pad12) -> DISP_PWM
- U5 pad 40: Net-(U5-Pad40) -> DISP_PWM_POT
- U5 pad 41: Net-(U5-Pad41) -> R_JOYSTICK_BTN
- U5 pad 8: Net-(U5-Pad8) -> L_JOYSTICK_BTN
