File: hdmi.sch (KiCad schematic (older format))
At the start: 12 parts

Commit message: Wired up the DPI display and Camera
Still need to wire up the DPI connector.
Connections:
- net GND: now also Q?.2 (S)
Changed lines of the file:
@@
 Text Notes 6800 1150 0    100  ~ 0
 VERIFY THIS COMPONENT
+Wire Wire Line
+	10300 4200 10300 4400
+$Comp
+L power:GND #PWR?
+U 1 1 5EC02BE0
+P 10300 4400
+F 0 "#PWR?" H 10300 4150 50  0001 C CNN
+F 1 "GND" H 10305 4227 50  0000 C CNN
+F 2 "" H 10300 4400 50  0001 C CNN
+F 3 "" H 10300 4400 50  0001 C CNN
+	1    10300 4400
+	1    0    0    -1
+$EndComp
 $EndSCHEMATC

Commit message: Added USB Ports and wired up more of the DPI connector
Parts:
- C19: renamed from C?; footprint (none) -> Capacitor_SMD:C_0805_2012Metric
- J9: renamed from J?; footprint digikey-footprints:HDMI_Mini_Female_2001-1-2-21-00-BK -> Connector_HDMI:HDMI_Micro-D_Molex_46765-2x0x
- MD1: renamed from MD?; footprint _ -> footprints:Conn_TE-DDR2-SODIMM-0.6-200P-doublesided
- R19, R20, R21: renamed from R?; footprint (none) -> Resistor_SMD:R_0805_2012Metric
- gave numbers to parts that had none: 6
Changed lines of the file:
@@
 $EndDescr
 $Comp
-L dk_USB-DVI-HDMI-Connectors:2001-1-2-21-00-BK J?
+L dk_USB-DVI-HDMI-Connectors:2001-1-2-21-00-BK J9
 U 1 1 5EBB29FE
 P 5350 2600
-F 0 "J?" H 5488 4232 60  0000 C CNN
+F 0 "J9" H 5488 4232 60  0000 C CNN
 F 1 "2001-1-2-21-00-BK" H 5488 4126 60  0000 C CNN
-F 2 "digikey-footprints:HDMI_Mini_Female_2001-1-2-21-00-BK" H 5550 2800 60  0001 L CNN
+F 2 "Connector_HDMI:HDMI_Micro-D_Molex_46765-2x0x" H 5550 2800 60  0001 L CNN
 F 3 "http://cnctech.us/pdfs/2001-1-2-21-00-BK.pdf" H 5550 2900 60  0001 L CNN
 F 4 "1175-1704-1-ND" H 5550 3000 60  0001 L CNN "Digi-Key_PN"
@@
 HDMI_CEC
 $Comp
-L KiCADinfo_RPi-modules:Board_RPi_CM3lite_200pConnector_multipart MD?
+L KiCADinfo_RPi-modules:Board_RPi_CM3lite_200pConnector_multipart MD1
 U 4 1 5EBAF503
 P 2600 2600
-F 0 "MD?" H 2683 3875 50  0000 C CNN
+F 0 "MD1" H 2683 3875 50  0000 C CNN
 F 1 "Board_RPi_CM3lite_200pConnector_multipart" H 2683 3784 50  0000 C CNN
-F 2 "_" H 8575 -250 10  0001 C CNN
+F 2 "footprints:Conn_TE-DDR2-SODIMM-0.6-200P-doublesided" H 8575 -250 10  0001 C CNN
 F 3 "_" H 8575 -250 10  0001 C CNN
 F 4 "_" H 8575 -250 10  0001 C CNN "Manf#"
@@
 	6050 3300 6050 4100
 $Comp
-L power:GND #PWR?
+L power:GND #PWR0174
 U 1 1 5EBCDFD6
 P 5250 4100
-F 0 "#PWR?" H 5250 3850 50  0001 C CNN
+F 0 "#PWR0174" H 5250 3850 50  0001 C CNN
 F 1 "GND" H 5255 3927 50  0000 C CNN
 F 2 "" H 5250 4100 50  0001 C CNN
@@
 $EndComp
 $Comp
-L power:GND #PWR?
+L power:GND #PWR0175
 U 1 1 5EBCEB52
 P 6050 4100
-F 0 "#PWR?" H 6050 3850 50  0001 C CNN
+F 0 "#PWR0175" H 6050 3850 50  0001 C CNN
 F 1 "GND" H 6055 3927 50  0000 C CNN
 F 2 "" H 6050 4100 50  0001 C CNN
@@
 	5950 3400 6550 3400
 $Comp
-L Device:C C?
+L Device:C C19
 U 1 1 5EBCF7BE
 P 6550 3800
-F 0 "C?" H 6665 3846 50  0000 L CNN
+F 0 "C19" H 6665 3846 50  0000 L CNN
 F 1 "C" H 6665 3755 50  0000 L CNN
-F 2 "" H 6588 3650 50  0001 C CNN
+F 2 "Capacitor_SMD:C_0805_2012Metric" H 6588 3650 50  0001 C CNN
 F 3 "~" H 6550 3800 50  0001 C CNN
 	1    6550 3800
@@
 $EndComp
 $Comp
-L power:GND #PWR?
+L power:GND #PWR0176
 U 1 1 5EBD0798
 P 6550 4100
-F 0 "#PWR?" H 6550 3850 50  0001 C CNN
+F 0 "#PWR0176" H 6550 3850 50  0001 C CNN
 F 1 "GND" H 6555 3927 50  0000 C CNN
 F 2 "" H 6550 4100 50  0001 C CNN
@@
 	6550 3650 6550 3400
 $Comp
-L Diode:BAV99 D?
+L Diode:BAV99 D4
 U 1 1 5EBD1C7B
 P 7550 4000
-F 0 "D?" V 7596 4079 50  0000 L CNN
+F 0 "D4" V 7596 4079 50  0000 L CNN
 F 1 "BAV99" V 7505 4079 50  0000 L CNN
 F 2 "Package_TO_SOT_SMD:SOT-23" H 7550 3500 50  0001 C CNN
@@
 $EndComp
 $Comp
-L Diode:BAV99 D?
+L Diode:BAV99 D5
 U 1 1 5EBD575A
 P 8200 4000
-F 0 "D?" V 8246 4079 50  0000 L CNN
+F 0 "D5" V 8246 4079 50  0000 L CNN
 F 1 "BAV99" V 8155 4079 50  0000 L CNN
 F 2 "Package_TO_SOT_SMD:SOT-23" H 8200 3500 50  0001 C CNN
@@
 $EndComp
 $Comp
-L Diode:BAV99 D?
+L Diode:BAV99 D6
 U 1 1 5EBD5CB0
 P 8850 4000
-F 0 "D?" V 8896 4079 50  0000 L CNN
+F 0 "D6" V 8896 4079 50  0000 L CNN
 F 1 "BAV99" V 8805 4079 50  0000 L CNN
 F 2 "Package_TO_SOT_SMD:SOT-23" H 8850 3500 50  0001 C CNN
@@
 $EndComp
 $Comp
-L Diode:BAV99 D?
+L Diode:BAV99 D7
 U 1 1 5EBD61ED
 P 9500 4000
-F 0 "D?" V 9546 4079 50  0000 L CNN
+F 0 "D7" V 9546 4079 50  0000 L CNN
 F 1 "BAV99" V 9455 4079 50  0000 L CNN
 F 2 "Package_TO_SOT_SMD:SOT-23" H 9500 3500 50  0001 C CNN
@@
 $EndComp
 $Comp
-L Transistor_FET:2N7002 Q?
+L Transistor_FET:2N7002 Q1
 U 1 1 5EBD6B28
 P 10200 4000
-F 0 "Q?" H 10405 4046 50  0000 L CNN
+F 0 "Q1" H 10405 4046 50  0000 L CNN
 F 1 "2N7002P.215" H 10405 3955 50  0000 L CNN
 F 2 "Package_TO_SOT_SMD:SOT-23" H 10400 3925 50  0001 L CIN
@@
 $EndComp
 $Comp
-L Device:R R?
+L Device:R R21
 U 1 1 5EBDB81D
 P 10300 3500
-F 0 "R?" H 10370 3546 50  0000 L CNN
+F 0 "R21" H 10370 3546 50  0000 L CNN
 F 1 "100k" V 10300 3400 50  0000 L CNN
-F 2 "" V 10230 3500 50  0001 C CNN
+F 2 "Resistor_SMD:R_0805_2012Metric" V 10230 3500 50  0001 C CNN
 F 3 "~" H 10300 3500 50  0001 C CNN
 	1    10300 3500
@@
 	7550 3700 7550 1950
 $Comp
-L power:+3V3 #PWR?
+L power:+3V3 #PWR0177
 U 1 1 5EBEB986
 P 7550 1950
-F 0 "#PWR?" H 7550 1800 50  0001 C CNN
+F 0 "#PWR0177" H 7550 1800 50  0001 C CNN
 F 1 "+3V3" H 7565 2123 50  0000 C CNN
 F 2 "" H 7550 1950 50  0001 C CNN
@@
 $EndComp
 $Comp
-L power:GND #PWR?
+L power:GND #PWR0178
 U 1 1 5EBEBF92
 P 7550 4400
-F 0 "#PWR?" H 7550 4150 50  0001 C CNN
+F 0 "#PWR0178" H 7550 4150 50  0001 C CNN
 F 1 "GND" H 7555 4227 50  0000 C CNN
 F 2 "" H 7550 4400 50  0001 C CNN
@@
 $EndComp
 $Comp
-L power:GND #PWR?
+L power:GND #PWR0179
 U 1 1 5EBEC5BD
 P 8200 4400
-F 0 "#PWR?" H 8200 4150 50  0001 C CNN
+F 0 "#PWR0179" H 8200 4150 50  0001 C CNN
 F 1 "GND" H 8205 4227 50  0000 C CNN
 F 2 "" H 8200 4400 50  0001 C CNN
@@
 $EndComp
 $Comp
-L power:GND #PWR?
+L power:GND #PWR0180
 U 1 1 5EBEC7F1
 P 8850 4400
-F 0 "#PWR?" H 8850 4150 50  0001 C CNN
+F 0 "#PWR0180" H 8850 4150 50  0001 C CNN
 F 1 "GND" H 8855 4227 50  0000 C CNN
 F 2 "" H 8850 4400 50  0001 C CNN
@@
 $EndComp
 $Comp
-L power:GND #PWR?
+L power:GND #PWR0181
 U 1 1 5EBECAA3
 P 9500 4400
-F 0 "#PWR?" H 9500 4150 50  0001 C CNN
+F 0 "#PWR0181" H 9500 4150 50  0001 C CNN
 F 1 "GND" H 9505 4227 50  0000 C CNN
 F 2 "" H 9500 4400 50  0001 C CNN
@@
 	8600 3200 8600 2450
 $Comp
-L Device:R R?
+L Device:R R19
 U 1 1 5EBF2D57
 P 7950 2300
-F 0 "R?" H 8020 2346 50  0000 L CNN
+F 0 "R19" H 8020 2346 50  0000 L CNN
 F 1 "1.8k" V 7950 2200 50  0000 L CNN
-F 2 "" V 7880 2300 50  0001 C CNN
+F 2 "Resistor_SMD:R_0805_2012Metric" V 7880 2300 50  0001 C CNN
 F 3 "~" H 7950 2300 50  0001 C CNN
 	1    7950 2300
@@
 $EndComp
 $Comp
-L Device:R R?
+L Device:R R20
 U 1 1 5EBF3577
 P 8600 2300
-F 0 "R?" H 8670 2346 50  0000 L CNN
+F 0 "R20" H 8670 2346 50  0000 L CNN
 F 1 "1.8k" V 8600 2200 50  0000 L CNN
-F 2 "" V 8530 2300 50  0001 C CNN
+F 2 "Resistor_SMD:R_0805_2012Metric" V 8530 2300 50  0001 C CNN
 F 3 "~" H 8600 2300 50  0001 C CNN
 	1    8600 2300
@@
 	7050 3400 6550 3400
 $Comp
-L power:+5V #PWR?
+L power:+5V #PWR0182
 U 1 1 5EBF7F39
 P 7950 1950
-F 0 "#PWR?" H 7950 1800 50  0001 C CNN
+F 0 "#PWR0182" H 7950 1800 50  0001 C CNN
 F 1 "+5V" H 7965 2123 50  0000 C CNN
 F 2 "" H 7950 1950 50  0001 C CNN
@@
 $EndComp
 $Comp
-L power:+5V #PWR?
+L power:+5V #PWR0183
 U 1 1 5EBF86C5
 P 8600 1950
-F 0 "#PWR?" H 8600 1800 50  0001 C CNN
+F 0 "#PWR0183" H 8600 1800 50  0001 C CNN
 F 1 "+5V" H 8615 2123 50  0000 C CNN
 F 2 "" H 8600 1950 50  0001 C CNN
@@
 $EndComp
 $Comp
-L Diode:BAT54A D?
+L Diode:BAT54A D3
 U 1 1 5EBFC4A3
 P 7050 1500
-F 0 "D?" V 7004 1588 50  0000 L CNN
+F 0 "D3" V 7004 1588 50  0000 L CNN
 F 1 "BAT54A" V 7095 1588 50  0000 L CNN
 F 2 "Package_TO_SOT_SMD:SOT-23" H 7125 1625 50  0001 L CNN
@@
 	6700 1500 6700 850
 $Comp
-L power:+5V #PWR?
+L power:+5V #PWR0184
 U 1 1 5EBFFBEB
 P 6700 850
-F 0 "#PWR?" H 6700 700 50  0001 C CNN
+F 0 "#PWR0184" H 6700 700 50  0001 C CNN
 F 1 "+5V" H 6715 1023 50  0000 C CNN
 F 2 "" H 6700 850 50  0001 C CNN
@@
 	10300 4200 10300 4400
 $Comp
-L power:GND #PWR?
+L power:GND #PWR0185
 U 1 1 5EC02BE0
 P 10300 4400
-F 0 "#PWR?" H 10300 4150 50  0001 C CNN
+F 0 "#PWR0185" H 10300 4150 50  0001 C CNN
 F 1 "GND" H 10305 4227 50  0000 C CNN
 F 2 "" H 10300 4400 50  0001 C CNN

Commit message: Added documentation
Parts:
- renumbered C19 to C26, D6 to D10, D7 to D11, D3 to D7, D4 to D8, D5 to D9, J9 to J11, R19 to R27, R20 to R28, R21 to R29
Changed lines of the file:
@@
 $EndDescr
 $Comp
-L dk_USB-DVI-HDMI-Connectors:2001-1-2-21-00-BK J9
+L dk_USB-DVI-HDMI-Connectors:2001-1-2-21-00-BK J11
 U 1 1 5EBB29FE
 P 5350 2600
-F 0 "J9" H 5488 4232 60  0000 C CNN
+F 0 "J11" H 5488 4232 60  0000 C CNN
 F 1 "2001-1-2-21-00-BK" H 5488 4126 60  0000 C CNN
 F 2 "Connector_HDMI:HDMI_Micro-D_Molex_46765-2x0x" H 5550 2800 60  0001 L CNN
@@
 	6050 3300 6050 4100
 $Comp
-L power:GND #PWR0174
+L power:GND #PWR0101
 U 1 1 5EBCDFD6
 P 5250 4100
-F 0 "#PWR0174" H 5250 3850 50  0001 C CNN
+F 0 "#PWR0101" H 5250 3850 50  0001 C CNN
 F 1 "GND" H 5255 3927 50  0000 C CNN
 F 2 "" H 5250 4100 50  0001 C CNN
@@
 $EndComp
 $Comp
-L power:GND #PWR0175
+L power:GND #PWR0102
 U 1 1 5EBCEB52
 P 6050 4100
-F 0 "#PWR0175" H 6050 3850 50  0001 C CNN
+F 0 "#PWR0102" H 6050 3850 50  0001 C CNN
 F 1 "GND" H 6055 3927 50  0000 C CNN
 F 2 "" H 6050 4100 50  0001 C CNN
@@
 	5950 3400 6550 3400
 $Comp
-L Device:C C19
+L Device:C C26
 U 1 1 5EBCF7BE
 P 6550 3800
-F 0 "C19" H 6665 3846 50  0000 L CNN
+F 0 "C26" H 6665 3846 50  0000 L CNN
 F 1 "C" H 6665 3755 50  0000 L CNN
 F 2 "Capacitor_SMD:C_0805_2012Metric" H 6588 3650 50  0001 C CNN
@@
 $EndComp
 $Comp
-L power:GND #PWR0176
+L power:GND #PWR0103
 U 1 1 5EBD0798
 P 6550 4100
-F 0 "#PWR0176" H 6550 3850 50  0001 C CNN
+F 0 "#PWR0103" H 6550 3850 50  0001 C CNN
 F 1 "GND" H 6555 3927 50  0000 C CNN
 F 2 "" H 6550 4100 50  0001 C CNN
@@
 	6550 3650 6550 3400
 $Comp
-L Diode:BAV99 D4
+L Diode:BAV99 D8
 U 1 1 5EBD1C7B
 P 7550 4000
-F 0 "D4" V 7596 4079 50  0000 L CNN
+F 0 "D8" V 7596 4079 50  0000 L CNN
 F 1 "BAV99" V 7505 4079 50  0000 L CNN
 F 2 "Package_TO_SOT_SMD:SOT-23" H 7550 3500 50  0001 C CNN
@@
 $EndComp
 $Comp
-L Diode:BAV99 D5
+L Diode:BAV99 D9
 U 1 1 5EBD575A
 P 8200 4000
-F 0 "D5" V 8246 4079 50  0000 L CNN
+F 0 "D9" V 8246 4079 50  0000 L CNN
 F 1 "BAV99" V 8155 4079 50  0000 L CNN
 F 2 "Package_TO_SOT_SMD:SOT-23" H 8200 3500 50  0001 C CNN
@@
 $EndComp
 $Comp
-L Diode:BAV99 D6
+L Diode:BAV99 D10
 U 1 1 5EBD5CB0
 P 8850 4000
-F 0 "D6" V 8896 4079 50  0000 L CNN
+F 0 "D10" V 8896 4079 50  0000 L CNN
 F 1 "BAV99" V 8805 4079 50  0000 L CNN
 F 2 "Package_TO_SOT_SMD:SOT-23" H 8850 3500 50  0001 C CNN
@@
 $EndComp
 $Comp
-L Diode:BAV99 D7
+L Diode:BAV99 D11
 U 1 1 5EBD61ED
 P 9500 4000
-F 0 "D7" V 9546 4079 50  0000 L CNN
+F 0 "D11" V 9546 4079 50  0000 L CNN
 F 1 "BAV99" V 9455 4079 50  0000 L CNN
 F 2 "Package_TO_SOT_SMD:SOT-23" H 9500 3500 50  0001 C CNN
@@
 $EndComp
 $Comp
-L Device:R R21
+L Device:R R29
 U 1 1 5EBDB81D
 P 10300 3500
-F 0 "R21" H 10370 3546 50  0000 L CNN
+F 0 "R29" H 10370 3546 50  0000 L CNN
 F 1 "100k" V 10300 3400 50  0000 L CNN
 F 2 "Resistor_SMD:R_0805_2012Metric" V 10230 3500 50  0001 C CNN
@@
 	7550 3700 7550 1950
 $Comp
-L power:+3V3 #PWR0177
+L power:+3V3 #PWR0105
 U 1 1 5EBEB986
 P 7550 1950
-F 0 "#PWR0177" H 7550 1800 50  0001 C CNN
+F 0 "#PWR0105" H 7550 1800 50  0001 C CNN
 F 1 "+3V3" H 7565 2123 50  0000 C CNN
 F 2 "" H 7550 1950 50  0001 C CNN
@@
 $EndComp
 $Comp
-L power:GND #PWR0178
+L power:GND #PWR0106
 U 1 1 5EBEBF92
 P 7550 4400
-F 0 "#PWR0178" H 7550 4150 50  0001 C CNN
+F 0 "#PWR0106" H 7550 4150 50  0001 C CNN
 F 1 "GND" H 7555 4227 50  0000 C CNN
 F 2 "" H 7550 4400 50  0001 C CNN
@@
 $EndComp
 $Comp
-L power:GND #PWR0179
+L power:GND #PWR0108
 U 1 1 5EBEC5BD
 P 8200 4400
-F 0 "#PWR0179" H 8200 4150 50  0001 C CNN
+F 0 "#PWR0108" H 8200 4150 50  0001 C CNN
 F 1 "GND" H 8205 4227 50  0000 C CNN
 F 2 "" H 8200 4400 50  0001 C CNN
@@
 $EndComp
 $Comp
-L power:GND #PWR0180
+L power:GND #PWR0110
 U 1 1 5EBEC7F1
 P 8850 4400
-F 0 "#PWR0180" H 8850 4150 50  0001 C CNN
+F 0 "#PWR0110" H 8850 4150 50  0001 C CNN
 F 1 "GND" H 8855 4227 50  0000 C CNN
 F 2 "" H 8850 4400 50  0001 C CNN
@@
 $EndComp
 $Comp
-L power:GND #PWR0181
+L power:GND #PWR0111
 U 1 1 5EBECAA3
 P 9500 4400
-F 0 "#PWR0181" H 9500 4150 50  0001 C CNN
+F 0 "#PWR0111" H 9500 4150 50  0001 C CNN
 F 1 "GND" H 9505 4227 50  0000 C CNN
 F 2 "" H 9500 4400 50  0001 C CNN
@@
 	8600 3200 8600 2450
 $Comp
-L Device:R R19
+L Device:R R27
 U 1 1 5EBF2D57
 P 7950 2300
-F 0 "R19" H 8020 2346 50  0000 L CNN
+F 0 "R27" H 8020 2346 50  0000 L CNN
 F 1 "1.8k" V 7950 2200 50  0000 L CNN
 F 2 "Resistor_SMD:R_0805_2012Metric" V 7880 2300 50  0001 C CNN
@@
 $EndComp
 $Comp
-L Device:R R20
+L Device:R R28
 U 1 1 5EBF3577
 P 8600 2300
-F 0 "R20" H 8670 2346 50  0000 L CNN
+F 0 "R28" H 8670 2346 50  0000 L CNN
 F 1 "1.8k" V 8600 2200 50  0000 L CNN
 F 2 "Resistor_SMD:R_0805_2012Metric" V 8530 2300 50  0001 C CNN
@@
 	7050 3400 6550 3400
 $Comp
-L power:+5V #PWR0182
+L power:+5V #PWR0107
 U 1 1 5EBF7F39
 P 7950 1950
-F 0 "#PWR0182" H 7950 1800 50  0001 C CNN
+F 0 "#PWR0107" H 7950 1800 50  0001 C CNN
 F 1 "+5V" H 7965 2123 50  0000 C CNN
 F 2 "" H 7950 1950 50  0001 C CNN
@@
 $EndComp
 $Comp
-L power:+5V #PWR0183
+L power:+5V #PWR0109
 U 1 1 5EBF86C5
 P 8600 1950
-F 0 "#PWR0183" H 8600 1800 50  0001 C CNN
+F 0 "#PWR0109" H 8600 1800 50  0001 C CNN
 F 1 "+5V" H 8615 2123 50  0000 C CNN
 F 2 "" H 8600 1950 50  0001 C CNN
@@
 $EndComp
 $Comp
-L Diode:BAT54A D3
+L Diode:BAT54A D7
 U 1 1 5EBFC4A3
 P 7050 1500
-F 0 "D3" V 7004 1588 50  0000 L CNN
+F 0 "D7" V 7004 1588 50  0000 L CNN
 F 1 "BAT54A" V 7095 1588 50  0000 L CNN
 F 2 "Package_TO_SOT_SMD:SOT-23" H 7125 1625 50  0001 L CNN
@@
 	6700 1500 6700 850
 $Comp
-L power:+5V #PWR0184
+L power:+5V #PWR0104
 U 1 1 5EBFFBEB
 P 6700 850
-F 0 "#PWR0184" H 6700 700 50  0001 C CNN
+F 0 "#PWR0104" H 6700 700 50  0001 C CNN
 F 1 "+5V" H 6715 1023 50  0000 C CNN
 F 2 "" H 6700 850 50  0001 C CNN
@@
 	10300 4200 10300 4400
 $Comp
-L power:GND #PWR0185
+L power:GND #PWR0112
 U 1 1 5EC02BE0
 P 10300 4400
-F 0 "#PWR0185" H 10300 4150 50  0001 C CNN
+F 0 "#PWR0112" H 10300 4150 50  0001 C CNN
 F 1 "GND" H 10305 4227 50  0000 C CNN
 F 2 "" H 10300 4400 50  0001 C CNN

Commit message: Removed Second USB Hub
Also wired up a few more connections.
Parts:
- renumbered D7 to D5, D8 to D6, D9 to D7, D10 to D8, D11 to D9, R27 to R26, R28 to R27, R29 to R28
Changed lines of the file:
@@
 	6050 3300 6050 4100
 $Comp
-L power:GND #PWR0101
+L power:GND #PWR092
 U 1 1 5EBCDFD6
 P 5250 4100
-F 0 "#PWR0101" H 5250 3850 50  0001 C CNN
+F 0 "#PWR092" H 5250 3850 50  0001 C CNN
 F 1 "GND" H 5255 3927 50  0000 C CNN
 F 2 "" H 5250 4100 50  0001 C CNN
@@
 $EndComp
 $Comp
-L power:GND #PWR0102
+L power:GND #PWR093
 U 1 1 5EBCEB52
 P 6050 4100
-F 0 "#PWR0102" H 6050 3850 50  0001 C CNN
+F 0 "#PWR093" H 6050 3850 50  0001 C CNN
 F 1 "GND" H 6055 3927 50  0000 C CNN
 F 2 "" H 6050 4100 50  0001 C CNN
@@
 $EndComp
 $Comp
-L power:GND #PWR0103
+L power:GND #PWR094
 U 1 1 5EBD0798
 P 6550 4100
-F 0 "#PWR0103" H 6550 3850 50  0001 C CNN
+F 0 "#PWR094" H 6550 3850 50  0001 C CNN
 F 1 "GND" H 6555 3927 50  0000 C CNN
 F 2 "" H 6550 4100 50  0001 C CNN
@@
 	6550 3650 6550 3400
 $Comp
-L Diode:BAV99 D8
+L Diode:BAV99 D6
 U 1 1 5EBD1C7B
 P 7550 4000
-F 0 "D8" V 7596 4079 50  0000 L CNN
+F 0 "D6" V 7596 4079 50  0000 L CNN
 F 1 "BAV99" V 7505 4079 50  0000 L CNN
 F 2 "Package_TO_SOT_SMD:SOT-23" H 7550 3500 50  0001 C CNN
@@
 $EndComp
 $Comp
-L Diode:BAV99 D9
+L Diode:BAV99 D7
 U 1 1 5EBD575A
 P 8200 4000
-F 0 "D9" V 8246 4079 50  0000 L CNN
+F 0 "D7" V 8246 4079 50  0000 L CNN
 F 1 "BAV99" V 8155 4079 50  0000 L CNN
 F 2 "Package_TO_SOT_SMD:SOT-23" H 8200 3500 50  0001 C CNN
@@
 $EndComp
 $Comp
-L Diode:BAV99 D10
+L Diode:BAV99 D8
 U 1 1 5EBD5CB0
 P 8850 4000
-F 0 "D10" V 8896 4079 50  0000 L CNN
+F 0 "D8" V 8896 4079 50  0000 L CNN
 F 1 "BAV99" V 8805 4079 50  0000 L CNN
 F 2 "Package_TO_SOT_SMD:SOT-23" H 8850 3500 50  0001 C CNN
@@
 $EndComp
 $Comp
-L Diode:BAV99 D11
+L Diode:BAV99 D9
 U 1 1 5EBD61ED
 P 9500 4000
-F 0 "D11" V 9546 4079 50  0000 L CNN
+F 0 "D9" V 9546 4079 50  0000 L CNN
 F 1 "BAV99" V 9455 4079 50  0000 L CNN
 F 2 "Package_TO_SOT_SMD:SOT-23" H 9500 3500 50  0001 C CNN
@@
 $EndComp
 $Comp
-L Device:R R29
+L Device:R R28
 U 1 1 5EBDB81D
 P 10300 3500
-F 0 "R29" H 10370 3546 50  0000 L CNN
+F 0 "R28" H 10370 3546 50  0000 L CNN
 F 1 "100k" V 10300 3400 50  0000 L CNN
 F 2 "Resistor_SMD:R_0805_2012Metric" V 10230 3500 50  0001 C CNN
@@
 	7550 3700 7550 1950
 $Comp
-L power:+3V3 #PWR0105
+L power:+3V3 #PWR096
 U 1 1 5EBEB986
 P 7550 1950
-F 0 "#PWR0105" H 7550 1800 50  0001 C CNN
+F 0 "#PWR096" H 7550 1800 50  0001 C CNN
 F 1 "+3V3" H 7565 2123 50  0000 C CNN
 F 2 "" H 7550 1950 50  0001 C CNN
@@
 $EndComp
 $Comp
-L power:GND #PWR0106
+L power:GND #PWR097
 U 1 1 5EBEBF92
 P 7550 4400
-F 0 "#PWR0106" H 7550 4150 50  0001 C CNN
+F 0 "#PWR097" H 7550 4150 50  0001 C CNN
 F 1 "GND" H 7555 4227 50  0000 C CNN
 F 2 "" H 7550 4400 50  0001 C CNN
@@
 $EndComp
 $Comp
-L power:GND #PWR0108
+L power:GND #PWR099
 U 1 1 5EBEC5BD
 P 8200 4400
-F 0 "#PWR0108" H 8200 4150 50  0001 C CNN
+F 0 "#PWR099" H 8200 4150 50  0001 C CNN
 F 1 "GND" H 8205 4227 50  0000 C CNN
 F 2 "" H 8200 4400 50  0001 C CNN
@@
 $EndComp
 $Comp
-L power:GND #PWR0110
+L power:GND #PWR0101
 U 1 1 5EBEC7F1
 P 8850 4400
-F 0 "#PWR0110" H 8850 4150 50  0001 C CNN
+F 0 "#PWR0101" H 8850 4150 50  0001 C CNN
 F 1 "GND" H 8855 4227 50  0000 C CNN
 F 2 "" H 8850 4400 50  0001 C CNN
@@
 $EndComp
 $Comp
-L power:GND #PWR0111
+L power:GND #PWR0102
 U 1 1 5EBECAA3
 P 9500 4400
-F 0 "#PWR0111" H 9500 4150 50  0001 C CNN
+F 0 "#PWR0102" H 9500 4150 50  0001 C CNN
 F 1 "GND" H 9505 4227 50  0000 C CNN
 F 2 "" H 9500 4400 50  0001 C CNN
@@
 	8600 3200 8600 2450
 $Comp
-L Device:R R27
+L Device:R R26
 U 1 1 5EBF2D57
 P 7950 2300
-F 0 "R27" H 8020 2346 50  0000 L CNN
+F 0 "R26" H 8020 2346 50  0000 L CNN
 F 1 "1.8k" V 7950 2200 50  0000 L CNN
 F 2 "Resistor_SMD:R_0805_2012Metric" V 7880 2300 50  0001 C CNN
@@
 $EndComp
 $Comp
-L Device:R R28
+L Device:R R27
 U 1 1 5EBF3577
 P 8600 2300
-F 0 "R28" H 8670 2346 50  0000 L CNN
+F 0 "R27" H 8670 2346 50  0000 L CNN
 F 1 "1.8k" V 8600 2200 50  0000 L CNN
 F 2 "Resistor_SMD:R_0805_2012Metric" V 8530 2300 50  0001 C CNN
@@
 	7050 3400 6550 3400
 $Comp
-L power:+5V #PWR0107
+L power:+5V #PWR098
 U 1 1 5EBF7F39
 P 7950 1950
-F 0 "#PWR0107" H 7950 1800 50  0001 C CNN
+F 0 "#PWR098" H 7950 1800 50  0001 C CNN
 F 1 "+5V" H 7965 2123 50  0000 C CNN
 F 2 "" H 7950 1950 50  0001 C CNN
@@
 $EndComp
 $Comp
-L power:+5V #PWR0109
+L power:+5V #PWR0100
 U 1 1 5EBF86C5
 P 8600 1950
-F 0 "#PWR0109" H 8600 1800 50  0001 C CNN
+F 0 "#PWR0100" H 8600 1800 50  0001 C CNN
 F 1 "+5V" H 8615 2123 50  0000 C CNN
 F 2 "" H 8600 1950 50  0001 C CNN
@@
 $EndComp
 $Comp
-L Diode:BAT54A D7
+L Diode:BAT54A D5
 U 1 1 5EBFC4A3
 P 7050 1500
-F 0 "D7" V 7004 1588 50  0000 L CNN
+F 0 "D5" V 7004 1588 50  0000 L CNN
 F 1 "BAT54A" V 7095 1588 50  0000 L CNN
 F 2 "Package_TO_SOT_SMD:SOT-23" H 7125 1625 50  0001 L CNN
@@
 	6700 1500 6700 850
 $Comp
-L power:+5V #PWR0104
+L power:+5V #PWR095
 U 1 1 5EBFFBEB
 P 6700 850
-F 0 "#PWR0104" H 6700 700 50  0001 C CNN
+F 0 "#PWR095" H 6700 700 50  0001 C CNN
 F 1 "+5V" H 6715 1023 50  0000 C CNN
 F 2 "" H 6700 850 50  0001 C CNN
@@
 	10300 4200 10300 4400
 $Comp
-L power:GND #PWR0112
+L power:GND #PWR0103
 U 1 1 5EC02BE0
 P 10300 4400
-F 0 "#PWR0112" H 10300 4150 50  0001 C CNN
+F 0 "#PWR0103" H 10300 4150 50  0001 C CNN
 F 1 "GND" H 10305 4227 50  0000 C CNN
 F 2 "" H 10300 4400 50  0001 C CNN
