File: hdmi.sch (KiCad schematic (older format))
At the start: 12 parts, among them J11 2001-1-2-21-00-BK, Q1 2N7002P.215

Commit message: minor changes
Parts:
- renumbered C26 to C30, R26 to R24, R27 to R25, R28 to R26
Changed lines of the file:
@@
 	6050 3300 6050 4100
 $Comp
-L power:GND #PWR092
+L power:GND #PWR099
 U 1 1 5EBCDFD6
 P 5250 4100
-F 0 "#PWR092" H 5250 3850 50  0001 C CNN
+F 0 "#PWR099" H 5250 3850 50  0001 C CNN
 F 1 "GND" H 5255 3927 50  0000 C CNN
 F 2 "" H 5250 4100 50  0001 C CNN
@@
 $EndComp
 $Comp
-L power:GND #PWR093
+L power:GND #PWR0100
 U 1 1 5EBCEB52
 P 6050 4100
-F 0 "#PWR093" H 6050 3850 50  0001 C CNN
+F 0 "#PWR0100" H 6050 3850 50  0001 C CNN
 F 1 "GND" H 6055 3927 50  0000 C CNN
 F 2 "" H 6050 4100 50  0001 C CNN
@@
 	5950 3400 6550 3400
 $Comp
-L Device:C C26
+L Device:C C30
 U 1 1 5EBCF7BE
 P 6550 3800
-F 0 "C26" H 6665 3846 50  0000 L CNN
+F 0 "C30" H 6665 3846 50  0000 L CNN
 F 1 "C" H 6665 3755 50  0000 L CNN
 F 2 "Capacitor_SMD:C_0805_2012Metric" H 6588 3650 50  0001 C CNN
@@
 $EndComp
 $Comp
-L power:GND #PWR094
+L power:GND #PWR0101
 U 1 1 5EBD0798
 P 6550 4100
-F 0 "#PWR094" H 6550 3850 50  0001 C CNN
+F 0 "#PWR0101" H 6550 3850 50  0001 C CNN
 F 1 "GND" H 6555 3927 50  0000 C CNN
 F 2 "" H 6550 4100 50  0001 C CNN
@@
 $EndComp
 $Comp
-L Device:R R28
+L Device:R R26
 U 1 1 5EBDB81D
 P 10300 3500
-F 0 "R28" H 10370 3546 50  0000 L CNN
+F 0 "R26" H 10370 3546 50  0000 L CNN
 F 1 "100k" V 10300 3400 50  0000 L CNN
 F 2 "Resistor_SMD:R_0805_2012Metric" V 10230 3500 50  0001 C CNN
@@
 	7550 3700 7550 1950
 $Comp
-L power:+3V3 #PWR096
+L power:+3V3 #PWR0103
 U 1 1 5EBEB986
 P 7550 1950
-F 0 "#PWR096" H 7550 1800 50  0001 C CNN
+F 0 "#PWR0103" H 7550 1800 50  0001 C CNN
 F 1 "+3V3" H 7565 2123 50  0000 C CNN
 F 2 "" H 7550 1950 50  0001 C CNN
@@
 $EndComp
 $Comp
-L power:GND #PWR097
+L power:GND #PWR0104
 U 1 1 5EBEBF92
 P 7550 4400
-F 0 "#PWR097" H 7550 4150 50  0001 C CNN
+F 0 "#PWR0104" H 7550 4150 50  0001 C CNN
 F 1 "GND" H 7555 4227 50  0000 C CNN
 F 2 "" H 7550 4400 50  0001 C CNN
@@
 $EndComp
 $Comp
-L power:GND #PWR099
+L power:GND #PWR0106
 U 1 1 5EBEC5BD
 P 8200 4400
-F 0 "#PWR099" H 8200 4150 50  0001 C CNN
+F 0 "#PWR0106" H 8200 4150 50  0001 C CNN
 F 1 "GND" H 8205 4227 50  0000 C CNN
 F 2 "" H 8200 4400 50  0001 C CNN
@@
 $EndComp
 $Comp
-L power:GND #PWR0101
+L power:GND #PWR0108
 U 1 1 5EBEC7F1
 P 8850 4400
-F 0 "#PWR0101" H 8850 4150 50  0001 C CNN
+F 0 "#PWR0108" H 8850 4150 50  0001 C CNN
 F 1 "GND" H 8855 4227 50  0000 C CNN
 F 2 "" H 8850 4400 50  0001 C CNN
@@
 $EndComp
 $Comp
-L power:GND #PWR0102
+L power:GND #PWR0109
 U 1 1 5EBECAA3
 P 9500 4400
-F 0 "#PWR0102" H 9500 4150 50  0001 C CNN
+F 0 "#PWR0109" H 9500 4150 50  0001 C CNN
 F 1 "GND" H 9505 4227 50  0000 C CNN
 F 2 "" H 9500 4400 50  0001 C CNN
@@
 	8600 3200 8600 2450
 $Comp
-L Device:R R26
+L Device:R R24
 U 1 1 5EBF2D57
 P 7950 2300
-F 0 "R26" H 8020 2346 50  0000 L CNN
+F 0 "R24" H 8020 2346 50  0000 L CNN
 F 1 "1.8k" V 7950 2200 50  0000 L CNN
 F 2 "Resistor_SMD:R_0805_2012Metric" V 7880 2300 50  0001 C CNN
@@
 $EndComp
 $Comp
-L Device:R R27
+L Device:R R25
 U 1 1 5EBF3577
 P 8600 2300
-F 0 "R27" H 8670 2346 50  0000 L CNN
+F 0 "R25" H 8670 2346 50  0000 L CNN
 F 1 "1.8k" V 8600 2200 50  0000 L CNN
 F 2 "Resistor_SMD:R_0805_2012Metric" V 8530 2300 50  0001 C CNN
@@
 	7050 3400 6550 3400
 $Comp
-L power:+5V #PWR098
+L power:+5V #PWR0105
 U 1 1 5EBF7F39
 P 7950 1950
-F 0 "#PWR098" H 7950 1800 50  0001 C CNN
+F 0 "#PWR0105" H 7950 1800 50  0001 C CNN
 F 1 "+5V" H 7965 2123 50  0000 C CNN
 F 2 "" H 7950 1950 50  0001 C CNN
@@
 $EndComp
 $Comp
-L power:+5V #PWR0100
+L power:+5V #PWR0107
 U 1 1 5EBF86C5
 P 8600 1950
-F 0 "#PWR0100" H 8600 1800 50  0001 C CNN
+F 0 "#PWR0107" H 8600 1800 50  0001 C CNN
 F 1 "+5V" H 8615 2123 50  0000 C CNN
 F 2 "" H 8600 1950 50  0001 C CNN
@@
 	6700 1500 6700 850
 $Comp
-L power:+5V #PWR095
+L power:+5V #PWR0102
 U 1 1 5EBFFBEB
 P 6700 850
-F 0 "#PWR095" H 6700 700 50  0001 C CNN
+F 0 "#PWR0102" H 6700 700 50  0001 C CNN
 F 1 "+5V" H 6715 1023 50  0000 C CNN
 F 2 "" H 6700 850 50  0001 C CNN
@@
 	10300 4200 10300 4400
 $Comp
-L power:GND #PWR0103
+L power:GND #PWR0110
 U 1 1 5EC02BE0
 P 10300 4400
-F 0 "#PWR0103" H 10300 4150 50  0001 C CNN
+F 0 "#PWR0110" H 10300 4150 50  0001 C CNN
 F 1 "GND" H 10305 4227 50  0000 C CNN
 F 2 "" H 10300 4400 50  0001 C CNN

Commit message: Fixed footprints, added PWM to display backlight
Parts:
- J11: footprint Connector_HDMI:HDMI_Micro-D_Molex_46765-2x0x -> HDMI_MOLEX:HDMI_MOLEX_471510001
- renumbered D5 to D4, D6 to D5, D7 to D6, D8 to D7, D9 to D8, R24 to R22, R25 to R23, R26 to R24
Changed lines of the file:
@@
 F 0 "J11" H 5488 4232 60  0000 C CNN
 F 1 "2001-1-2-21-00-BK" H 5488 4126 60  0000 C CNN
-F 2 "Connector_HDMI:HDMI_Micro-D_Molex_46765-2x0x" H 5550 2800 60  0001 L CNN
+F 2 "HDMI_MOLEX:HDMI_MOLEX_471510001" H 5550 2800 60  0001 L CNN
 F 3 "http://cnctech.us/pdfs/2001-1-2-21-00-BK.pdf" H 5550 2900 60  0001 L CNN
 F 4 "1175-1704-1-ND" H 5550 3000 60  0001 L CNN "Digi-Key_PN"
@@
 	6050 3300 6050 4100
 $Comp
-L power:GND #PWR099
+L power:GND #PWR0100
 U 1 1 5EBCDFD6
 P 5250 4100
-F 0 "#PWR099" H 5250 3850 50  0001 C CNN
+F 0 "#PWR0100" H 5250 3850 50  0001 C CNN
 F 1 "GND" H 5255 3927 50  0000 C CNN
 F 2 "" H 5250 4100 50  0001 C CNN
@@
 $EndComp
 $Comp
-L power:GND #PWR0100
+L power:GND #PWR0101
 U 1 1 5EBCEB52
 P 6050 4100
-F 0 "#PWR0100" H 6050 3850 50  0001 C CNN
+F 0 "#PWR0101" H 6050 3850 50  0001 C CNN
 F 1 "GND" H 6055 3927 50  0000 C CNN
 F 2 "" H 6050 4100 50  0001 C CNN
@@
 $EndComp
 $Comp
-L power:GND #PWR0101
+L power:GND #PWR0102
 U 1 1 5EBD0798
 P 6550 4100
-F 0 "#PWR0101" H 6550 3850 50  0001 C CNN
+F 0 "#PWR0102" H 6550 3850 50  0001 C CNN
 F 1 "GND" H 6555 3927 50  0000 C CNN
 F 2 "" H 6550 4100 50  0001 C CNN
@@
 	6550 3650 6550 3400
 $Comp
-L Diode:BAV99 D6
+L Diode:BAV99 D5
 U 1 1 5EBD1C7B
 P 7550 4000
-F 0 "D6" V 7596 4079 50  0000 L CNN
+F 0 "D5" V 7596 4079 50  0000 L CNN
 F 1 "BAV99" V 7505 4079 50  0000 L CNN
 F 2 "Package_TO_SOT_SMD:SOT-23" H 7550 3500 50  0001 C CNN
@@
 $EndComp
 $Comp
-L Diode:BAV99 D7
+L Diode:BAV99 D6
 U 1 1 5EBD575A
 P 8200 4000
-F 0 "D7" V 8246 4079 50  0000 L CNN
+F 0 "D6" V 8246 4079 50  0000 L CNN
 F 1 "BAV99" V 8155 4079 50  0000 L CNN
 F 2 "Package_TO_SOT_SMD:SOT-23" H 8200 3500 50  0001 C CNN
@@
 $EndComp
 $Comp
-L Diode:BAV99 D8
+L Diode:BAV99 D7
 U 1 1 5EBD5CB0
 P 8850 4000
-F 0 "D8" V 8896 4079 50  0000 L CNN
+F 0 "D7" V 8896 4079 50  0000 L CNN
 F 1 "BAV99" V 8805 4079 50  0000 L CNN
 F 2 "Package_TO_SOT_SMD:SOT-23" H 8850 3500 50  0001 C CNN
@@
 $EndComp
 $Comp
-L Diode:BAV99 D9
+L Diode:BAV99 D8
 U 1 1 5EBD61ED
 P 9500 4000
-F 0 "D9" V 9546 4079 50  0000 L CNN
+F 0 "D8" V 9546 4079 50  0000 L CNN
 F 1 "BAV99" V 9455 4079 50  0000 L CNN
 F 2 "Package_TO_SOT_SMD:SOT-23" H 9500 3500 50  0001 C CNN
@@
 $EndComp
 $Comp
-L Device:R R26
+L Device:R R24
 U 1 1 5EBDB81D
 P 10300 3500
-F 0 "R26" H 10370 3546 50  0000 L CNN
+F 0 "R24" H 10370 3546 50  0000 L CNN
 F 1 "100k" V 10300 3400 50  0000 L CNN
 F 2 "Resistor_SMD:R_0805_2012Metric" V 10230 3500 50  0001 C CNN
@@
 	7550 3700 7550 1950
 $Comp
-L power:+3V3 #PWR0103
+L power:+3V3 #PWR0104
 U 1 1 5EBEB986
 P 7550 1950
-F 0 "#PWR0103" H 7550 1800 50  0001 C CNN
+F 0 "#PWR0104" H 7550 1800 50  0001 C CNN
 F 1 "+3V3" H 7565 2123 50  0000 C CNN
 F 2 "" H 7550 1950 50  0001 C CNN
@@
 $EndComp
 $Comp
-L power:GND #PWR0104
+L power:GND #PWR0105
 U 1 1 5EBEBF92
 P 7550 4400
-F 0 "#PWR0104" H 7550 4150 50  0001 C CNN
+F 0 "#PWR0105" H 7550 4150 50  0001 C CNN
 F 1 "GND" H 7555 4227 50  0000 C CNN
 F 2 "" H 7550 4400 50  0001 C CNN
@@
 $EndComp
 $Comp
-L power:GND #PWR0106
+L power:GND #PWR0107
 U 1 1 5EBEC5BD
 P 8200 4400
-F 0 "#PWR0106" H 8200 4150 50  0001 C CNN
+F 0 "#PWR0107" H 8200 4150 50  0001 C CNN
 F 1 "GND" H 8205 4227 50  0000 C CNN
 F 2 "" H 8200 4400 50  0001 C CNN
@@
 $EndComp
 $Comp
-L power:GND #PWR0108
+L power:GND #PWR0109
 U 1 1 5EBEC7F1
 P 8850 4400
-F 0 "#PWR0108" H 8850 4150 50  0001 C CNN
+F 0 "#PWR0109" H 8850 4150 50  0001 C CNN
 F 1 "GND" H 8855 4227 50  0000 C CNN
 F 2 "" H 8850 4400 50  0001 C CNN
@@
 $EndComp
 $Comp
-L power:GND #PWR0109
+L power:GND #PWR0110
 U 1 1 5EBECAA3
 P 9500 4400
-F 0 "#PWR0109" H 9500 4150 50  0001 C CNN
+F 0 "#PWR0110" H 9500 4150 50  0001 C CNN
 F 1 "GND" H 9505 4227 50  0000 C CNN
 F 2 "" H 9500 4400 50  0001 C CNN
@@
 	8600 3200 8600 2450
 $Comp
-L Device:R R24
+L Device:R R22
 U 1 1 5EBF2D57
 P 7950 2300
-F 0 "R24" H 8020 2346 50  0000 L CNN
+F 0 "R22" H 8020 2346 50  0000 L CNN
 F 1 "1.8k" V 7950 2200 50  0000 L CNN
 F 2 "Resistor_SMD:R_0805_2012Metric" V 7880 2300 50  0001 C CNN
@@
 $EndComp
 $Comp
-L Device:R R25
+L Device:R R23
 U 1 1 5EBF3577
 P 8600 2300
-F 0 "R25" H 8670 2346 50  0000 L CNN
+F 0 "R23" H 8670 2346 50  0000 L CNN
 F 1 "1.8k" V 8600 2200 50  0000 L CNN
 F 2 "Resistor_SMD:R_0805_2012Metric" V 8530 2300 50  0001 C CNN
@@
 	7050 3400 6550 3400
 $Comp
-L power:+5V #PWR0105
+L power:+5V #PWR0106
 U 1 1 5EBF7F39
 P 7950 1950
-F 0 "#PWR0105" H 7950 1800 50  0001 C CNN
+F 0 "#PWR0106" H 7950 1800 50  0001 C CNN
 F 1 "+5V" H 7965 2123 50  0000 C CNN
 F 2 "" H 7950 1950 50  0001 C CNN
@@
 $EndComp
 $Comp
-L power:+5V #PWR0107
+L power:+5V #PWR0108
 U 1 1 5EBF86C5
 P 8600 1950
-F 0 "#PWR0107" H 8600 1800 50  0001 C CNN
+F 0 "#PWR0108" H 8600 1800 50  0001 C CNN
 F 1 "+5V" H 8615 2123 50  0000 C CNN
 F 2 "" H 8600 1950 50  0001 C CNN
@@
 $EndComp
 $Comp
-L Diode:BAT54A D5
+L Diode:BAT54A D4
 U 1 1 5EBFC4A3
 P 7050 1500
-F 0 "D5" V 7004 1588 50  0000 L CNN
+F 0 "D4" V 7004 1588 50  0000 L CNN
 F 1 "BAT54A" V 7095 1588 50  0000 L CNN
 F 2 "Package_TO_SOT_SMD:SOT-23" H 7125 1625 50  0001 L CNN
@@
 	6700 1500 6700 850
 $Comp
-L power:+5V #PWR0102
+L power:+5V #PWR0103
 U 1 1 5EBFFBEB
 P 6700 850
-F 0 "#PWR0102" H 6700 700 50  0001 C CNN
+F 0 "#PWR0103" H 6700 700 50  0001 C CNN
 F 1 "+5V" H 6715 1023 50  0000 C CNN
 F 2 "" H 6700 850 50  0001 C CNN
@@
 	10300 4200 10300 4400
 $Comp
-L power:GND #PWR0110
+L power:GND #PWR0111
 U 1 1 5EC02BE0
 P 10300 4400
-F 0 "#PWR0110" H 10300 4150 50  0001 C CNN
+F 0 "#PWR0111" H 10300 4150 50  0001 C CNN
 F 1 "GND" H 10305 4227 50  0000 C CNN
 F 2 "" H 10300 4400 50  0001 C CNN

Commit message: Updated values for several parts
Mostly capacitors.  Still need to do further review the schematic before it's all the way finished.
Parts:
- renumbered C30 to C34, R22 to R24, R23 to R25, R24 to R26
Changed lines of the file:
@@
 	6050 3300 6050 4100
 $Comp
-L power:GND #PWR0100
+L power:GND #PWR0112
 U 1 1 5EBCDFD6
 P 5250 4100
-F 0 "#PWR0100" H 5250 3850 50  0001 C CNN
+F 0 "#PWR0112" H 5250 3850 50  0001 C CNN
 F 1 "GND" H 5255 3927 50  0000 C CNN
 F 2 "" H 5250 4100 50  0001 C CNN
@@
 $EndComp
 $Comp
-L power:GND #PWR0101
+L power:GND #PWR0113
 U 1 1 5EBCEB52
 P 6050 4100
-F 0 "#PWR0101" H 6050 3850 50  0001 C CNN
+F 0 "#PWR0113" H 6050 3850 50  0001 C CNN
 F 1 "GND" H 6055 3927 50  0000 C CNN
 F 2 "" H 6050 4100 50  0001 C CNN
@@
 	5950 3400 6550 3400
 $Comp
-L Device:C C30
+L Device:C C34
 U 1 1 5EBCF7BE
 P 6550 3800
-F 0 "C30" H 6665 3846 50  0000 L CNN
+F 0 "C34" H 6665 3846 50  0000 L CNN
 F 1 "C" H 6665 3755 50  0000 L CNN
 F 2 "Capacitor_SMD:C_0805_2012Metric" H 6588 3650 50  0001 C CNN
@@
 $EndComp
 $Comp
-L power:GND #PWR0102
+L power:GND #PWR0114
 U 1 1 5EBD0798
 P 6550 4100
-F 0 "#PWR0102" H 6550 3850 50  0001 C CNN
+F 0 "#PWR0114" H 6550 3850 50  0001 C CNN
 F 1 "GND" H 6555 3927 50  0000 C CNN
 F 2 "" H 6550 4100 50  0001 C CNN
@@
 $EndComp
 $Comp
-L Device:R R24
+L Device:R R26
 U 1 1 5EBDB81D
 P 10300 3500
-F 0 "R24" H 10370 3546 50  0000 L CNN
+F 0 "R26" H 10370 3546 50  0000 L CNN
 F 1 "100k" V 10300 3400 50  0000 L CNN
 F 2 "Resistor_SMD:R_0805_2012Metric" V 10230 3500 50  0001 C CNN
@@
 	7550 3700 7550 1950
 $Comp
-L power:+3V3 #PWR0104
+L power:+3V3 #PWR0116
 U 1 1 5EBEB986
 P 7550 1950
-F 0 "#PWR0104" H 7550 1800 50  0001 C CNN
+F 0 "#PWR0116" H 7550 1800 50  0001 C CNN
 F 1 "+3V3" H 7565 2123 50  0000 C CNN
 F 2 "" H 7550 1950 50  0001 C CNN
@@
 $EndComp
 $Comp
-L power:GND #PWR0105
+L power:GND #PWR0117
 U 1 1 5EBEBF92
 P 7550 4400
-F 0 "#PWR0105" H 7550 4150 50  0001 C CNN
+F 0 "#PWR0117" H 7550 4150 50  0001 C CNN
 F 1 "GND" H 7555 4227 50  0000 C CNN
 F 2 "" H 7550 4400 50  0001 C CNN
@@
 $EndComp
 $Comp
-L power:GND #PWR0107
+L power:GND #PWR0119
 U 1 1 5EBEC5BD
 P 8200 4400
-F 0 "#PWR0107" H 8200 4150 50  0001 C CNN
+F 0 "#PWR0119" H 8200 4150 50  0001 C CNN
 F 1 "GND" H 8205 4227 50  0000 C CNN
 F 2 "" H 8200 4400 50  0001 C CNN
@@
 $EndComp
 $Comp
-L power:GND #PWR0109
+L power:GND #PWR0121
 U 1 1 5EBEC7F1
 P 8850 4400
-F 0 "#PWR0109" H 8850 4150 50  0001 C CNN
+F 0 "#PWR0121" H 8850 4150 50  0001 C CNN
 F 1 "GND" H 8855 4227 50  0000 C CNN
 F 2 "" H 8850 4400 50  0001 C CNN
@@
 $EndComp
 $Comp
-L power:GND #PWR0110
+L power:GND #PWR0122
 U 1 1 5EBECAA3
 P 9500 4400
-F 0 "#PWR0110" H 9500 4150 50  0001 C CNN
+F 0 "#PWR0122" H 9500 4150 50  0001 C CNN
 F 1 "GND" H 9505 4227 50  0000 C CNN
 F 2 "" H 9500 4400 50  0001 C CNN
@@
 	8600 3200 8600 2450
 $Comp
-L Device:R R22
+L Device:R R24
 U 1 1 5EBF2D57
 P 7950 2300
-F 0 "R22" H 8020 2346 50  0000 L CNN
+F 0 "R24" H 8020 2346 50  0000 L CNN
 F 1 "1.8k" V 7950 2200 50  0000 L CNN
 F 2 "Resistor_SMD:R_0805_2012Metric" V 7880 2300 50  0001 C CNN
@@
 $EndComp
 $Comp
-L Device:R R23
+L Device:R R25
 U 1 1 5EBF3577
 P 8600 2300
-F 0 "R23" H 8670 2346 50  0000 L CNN
+F 0 "R25" H 8670 2346 50  0000 L CNN
 F 1 "1.8k" V 8600 2200 50  0000 L CNN
 F 2 "Resistor_SMD:R_0805_2012Metric" V 8530 2300 50  0001 C CNN
@@
 	7050 3400 6550 3400
 $Comp
-L power:+5V #PWR0106
+L power:+5V #PWR0118
 U 1 1 5EBF7F39
 P 7950 1950
-F 0 "#PWR0106" H 7950 1800 50  0001 C CNN
+F 0 "#PWR0118" H 7950 1800 50  0001 C CNN
 F 1 "+5V" H 7965 2123 50  0000 C CNN
 F 2 "" H 7950 1950 50  0001 C CNN
@@
 $EndComp
 $Comp
-L power:+5V #PWR0108
+L power:+5V #PWR0120
 U 1 1 5EBF86C5
 P 8600 1950
-F 0 "#PWR0108" H 8600 1800 50  0001 C CNN
+F 0 "#PWR0120" H 8600 1800 50  0001 C CNN
 F 1 "+5V" H 8615 2123 50  0000 C CNN
 F 2 "" H 8600 1950 50  0001 C CNN
@@
 	6700 1500 6700 850
 $Comp
-L power:+5V #PWR0103
+L power:+5V #PWR0115
 U 1 1 5EBFFBEB
 P 6700 850
-F 0 "#PWR0103" H 6700 700 50  0001 C CNN
+F 0 "#PWR0115" H 6700 700 50  0001 C CNN
 F 1 "+5V" H 6715 1023 50  0000 C CNN
 F 2 "" H 6700 850 50  0001 C CNN
@@
 	10300 4200 10300 4400
 $Comp
-L power:GND #PWR0111
+L power:GND #PWR0123
 U 1 1 5EC02BE0
 P 10300 4400
-F 0 "#PWR0111" H 10300 4150 50  0001 C CNN
+F 0 "#PWR0123" H 10300 4150 50  0001 C CNN
 F 1 "GND" H 10305 4227 50  0000 C CNN
 F 2 "" H 10300 4400 50  0001 C CNN

Commit message: Added more part values
Parts:
- C34: value C -> 10uF
Changed lines of the file:
@@
 P 6550 3800
 F 0 "C34" H 6665 3846 50  0000 L CNN
-F 1 "C" H 6665 3755 50  0000 L CNN
+F 1 "10uF" H 6665 3755 50  0000 L CNN
 F 2 "Capacitor_SMD:C_0805_2012Metric" H 6588 3650 50  0001 C CNN
 F 3 "~" H 6550 3800 50  0001 C CNN
